File: hardware/_autosave-AUDIO-BOARD.kicad_pcb (KiCad board)
At the start: 2 copper layers, 66 x 46 mm, 79 parts, among them J1 CON_USB_GCT_USB4105_REVA, J3 CON_USB_GCT_USB4105_REVA, J4 BATT, J5 SD-CARD-MEM2051-00-195-00-A, M1 MNT, M2 MNT, M3 MNT, M4 MNT, Q1 DMP2040USD-13, Q2 DMP2040USD-13, Q3 SI2324DS-T1-GE3, Q4 SI2324DS-T1-GE3, SW1 RST, U1 CS42L51-CNZ, U2 TLV73333PDBV, U3 STM32H725ZET6, U4 MCP73831-2-OT, Y1 12MHz

Commit message: update the design
Parts:
- moved Y1 4.42 mm to (159.2, 77.0)
Connections:
- U3 pad 25: Net-(C33-Pad1) -> Net-(C25-Pad1)
- U3 pad 26: Net-(C25-Pad1) -> Net-(C33-Pad1)
Changed lines of the file:
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@@
   )
   (footprint "Crystal:Crystal_SMD_3225-4Pin_3.2x2.5mm" (layer "F.Cu")
-    (at 156.25 73.75 90)
+    (at 159.25 77 90)
     (descr "SMD Crystal SERIES SMD3225/4 http://www.txccrystal.com/images/pdf/7m-accuracy.pdf, 3.2x2.5mm^2 package")
     (tags "SMD SMT crystal")
@@
       (net 90 "unconnected-(U3-Pad24)") (pinfunction "PF10") (pintype "bidirectional"))
     (pad "25" smd roundrect (at -10.6625 3.25) (size 1.475 0.3) (layers "F.Cu" "F.Paste" "F.Mask") (roundrect_rratio 0.25)
-      (net 36 "Net-(C33-Pad1)") (pinfunction "PH0-OSC_IN") (pintype "bidirectional"))
+      (net 34 "Net-(C25-Pad1)") (pinfunction "PH0-OSC_IN") (pintype "bidirectional"))
     (pad "26" smd roundrect (at -10.6625 3.75) (size 1.475 0.3) (layers "F.Cu" "F.Paste" "F.Mask") (roundrect_rratio 0.25)
-      (net 34 "Net-(C25-Pad1)") (pinfunction "PH1-OSC_OUT") (pintype "output"))
+      (net 36 "Net-(C33-Pad1)") (pinfunction "PH1-OSC_OUT") (pintype "output"))
     (pad "27" smd roundrect (at -10.6625 4.25) (size 1.475 0.3) (layers "F.Cu" "F.Paste" "F.Mask") (roundrect_rratio 0.25)
       (net 35 "Net-(C29-Pad1)") (pinfunction "NRST") (pintype "unspecified"))
