File: hardware/AUDIO-BOARD.kicad_sch (KiCad schematic)
At the start: 5 parts, among them J1 CON_USB_GCT_USB4105_REVA, J5 SD-CARD-MEM2051-00-195-00-A, M1 MNT, M2 MNT, M3 MNT

Commit message: Project setup
Other:
- added sheet PowerSupply (Power-Supply.kicad_sch)
- sheet Audio Codec: file audo-codec.kicad_sch -> audio-codec.kicad_sch
- moved on the sheet: J1, J5
Changed lines of the file:
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@@
 (kicad_sch (version 20211123) (generator eeschema)
   (paper "A4")
-  (wire (pts (xy 55.88 171.45) (xy 52.07 171.45))
+  (wire (pts (xy 52.07 160.02) (xy 48.26 160.02))
     (stroke (width 0) (type default) (color 0 0 0 0))
   )
-  (wire (pts (xy 55.88 175.26) (xy 55.88 171.45))
+  (wire (pts (xy 52.07 163.83) (xy 52.07 160.02))
     (stroke (width 0) (type default) (color 0 0 0 0))
   )
   (symbol (lib_id "Mechanical:MountingHole") (at 34.29 191.77 0) (unit 1)
-    (in_bom yes) (on_board yes) (fields_autoplaced)
+    (in_bom yes) (on_board yes)
     (property "Reference" "M3" (id 0) (at 36.83 190.4999 0)
       (effects (font (size 1.27 1.27)) (justify left))
@@
     )
   )
-  (symbol (lib_id "1KiCadLib:CON_USB_GCT_USB4105_REVA") (at 31.75 152.4 0) (unit 1)
+  (symbol (lib_id "1KiCadLib:CON_USB_GCT_USB4105_REVA") (at 27.94 140.97 0) (unit 1)
     (in_bom yes) (on_board yes) (fields_autoplaced)
-    (property "Reference" "J1" (id 0) (at 38.735 134.62 0))
-    (property "Value" "CON_USB_GCT_USB4105_REVA" (id 1) (at 38.735 137.16 0))
-    (property "Footprint" "1KiCadLib:CON_USB_GCT_USB4105_REVA" (id 2) (at 12.7 137.16 0)
+    (property "Reference" "J1" (id 0) (at 34.925 123.19 0))
+    (property "Value" "CON_USB_GCT_USB4105_REVA" (id 1) (at 34.925 125.73 0))
+    (property "Footprint" "1KiCadLib:CON_USB_GCT_USB4105_REVA" (id 2) (at 8.89 125.73 0)
       (effects (font (size 1.27 1.27)) (justify left bottom) hide)
     )
-    (property "Datasheet" "" (id 3) (at 31.75 152.4 0)
+    (property "Datasheet" "" (id 3) (at 27.94 140.97 0)
       (effects (font (size 1.27 1.27)) (justify left bottom) hide)
     )
-    (property "MAXIMUM_PACKAGE_HEIGHT" "3.31 mm" (id 4) (at 25.4 146.05 0)
+    (property "MAXIMUM_PACKAGE_HEIGHT" "3.31 mm" (id 4) (at 21.59 134.62 0)
       (effects (font (size 1.27 1.27)) (justify left bottom) hide)
     )
-    (property "MANUFACTURER" "GCT" (id 5) (at 31.75 152.4 0)
+    (property "MANUFACTURER" "GCT" (id 5) (at 27.94 140.97 0)
       (effects (font (size 1.27 1.27)) (justify left bottom) hide)
     )
-    (property "PARTREV" "0.2" (id 6) (at 31.75 152.4 0)
+    (property "PARTREV" "0.2" (id 6) (at 27.94 140.97 0)
       (effects (font (size 1.27 1.27)) (justify left bottom) hide)
     )
-    (property "STANDARD" "Manufacturer Recommendations" (id 7) (at 13.97 134.62 0)
+    (property "STANDARD" "Manufacturer Recommendations" (id 7) (at 10.16 123.19 0)
       (effects (font (size 1.27 1.27)) (justify left bottom) hide)
     )
@@
     (pin "G4")
   )
-  (symbol (lib_id "power:GND") (at 55.88 175.26 0) (unit 1)
+  (symbol (lib_id "power:GND") (at 52.07 163.83 0) (unit 1)
     (in_bom yes) (on_board yes)
-    (property "Reference" "#PWR0103" (id 0) (at 55.88 181.61 0)
+    (property "Reference" "#PWR0103" (id 0) (at 52.07 170.18 0)
       (effects (font (size 1.27 1.27)) hide)
     )
-    (property "Value" "GND" (id 1) (at 59.69 176.53 0))
-    (property "Footprint" "" (id 2) (at 55.88 175.26 0)
+    (property "Value" "GND" (id 1) (at 55.88 165.1 0))
+    (property "Footprint" "" (id 2) (at 52.07 163.83 0)
       (effects (font (size 1.27 1.27)) hide)
     )
-    (property "Datasheet" "" (id 3) (at 55.88 175.26 0)
+    (property "Datasheet" "" (id 3) (at 52.07 163.83 0)
       (effects (font (size 1.27 1.27)) hide)
     )
@@
   )
   (symbol (lib_id "Mechanical:MountingHole") (at 25.4 191.77 0) (unit 1)
-    (in_bom yes) (on_board yes) (fields_autoplaced)
+    (in_bom yes) (on_board yes)
     (property "Reference" "M2" (id 0) (at 27.94 190.4999 0)
       (effects (font (size 1.27 1.27)) (justify left))
@@
     )
   )
-  (symbol (lib_id "1KiCadLib:SD-CARD-MEM2051-00-195-00-A") (at 224.79 143.51 0) (unit 1)
+  (symbol (lib_id "1KiCadLib:SD-CARD-MEM2051-00-195-00-A") (at 229.87 119.38 0) (unit 1)
     (in_bom yes) (on_board yes) (fields_autoplaced)
-    (property "Reference" "J5" (id 0) (at 224.79 128.27 0))
-    (property "Value" "SD-CARD-MEM2051-00-195-00-A" (id 1) (at 224.79 130.81 0))
-    (property "Footprint" "1KiCadLib:SD-CARD-MEM2051-00-195-00-A" (id 2) (at 222.25 128.27 0)
+    (property "Reference" "J5" (id 0) (at 229.87 104.14 0))
+    (property "Value" "SD-CARD-MEM2051-00-195-00-A" (id 1) (at 229.87 106.68 0))
+    (property "Footprint" "1KiCadLib:SD-CARD-MEM2051-00-195-00-A" (id 2) (at 227.33 104.14 0)
       (effects (font (size 1.27 1.27)) (justify bottom) hide)
     )
-    (property "Datasheet" "https://www.mouser.fr/ProductDetail/GCT/MEM2051-00-195-00-A?qs=KUoIvG%2F9Ilat7yfJRNWXUQ%3D%3D" (id 3) (at 224.79 129.54 0)
+    (property "Datasheet" "https://www.mouser.fr/ProductDetail/GCT/MEM2051-00-195-00-A?qs=KUoIvG%2F9Ilat7yfJRNWXUQ%3D%3D" (id 3) (at 229.87 105.41 0)
       (effects (font (size 1.27 1.27)) hide)
     )
-    (property "Manufacturer" "GCT" (id 4) (at 224.79 143.51 0)
+    (property "Manufacturer" "GCT" (id 4) (at 229.87 119.38 0)
       (effects (font (size 1.27 1.27)) (justify bottom) hide)
     )
-    (property "MPN" "MEM2051-00-195-00-A" (id 5) (at 220.98 121.92 0)
+    (property "MPN" "MEM2051-00-195-00-A" (id 5) (at 226.06 97.79 0)
       (effects (font (size 1.27 1.27)) hide)
     )
-    (property "Mouser" "640-MEM20510019500A" (id 6) (at 219.71 124.46 0)
+    (property "Mouser" "640-MEM20510019500A" (id 6) (at 224.79 100.33 0)
       (effects (font (size 1.27 1.27)) hide)
     )
@@
     (pin "9")
   )
-  (sheet (at 163.83 43.18) (size 44.45 25.4) (fields_autoplaced)
+  (sheet (at 198.12 29.21) (size 58.42 40.64) (fields_autoplaced)
     (stroke (width 0.1524) (type solid) (color 128 77 0 1))
     (fill (color 255 255 194 1.0000))
-    (property "Sheet name" "Audio Codec" (id 0) (at 163.83 42.4684 0)
+    (property "Sheet name" "Audio Codec" (id 0) (at 198.12 28.4984 0)
       (effects (font (size 1.27 1.27)) (justify left bottom))
     )
-    (property "Sheet file" "audo-codec.kicad_sch" (id 1) (at 163.83 69.1646 0)
+    (property "Sheet file" "audio-codec.kicad_sch" (id 1) (at 198.12 70.4346 0)
+      (effects (font (size 1.27 1.27)) (justify left top))
+    )
+  )
+  (sheet (at 27.94 25.4) (size 80.01 43.18) (fields_autoplaced)
+    (stroke (width 0.1524) (type solid) (color 0 0 0 0))
+    (fill (color 0 0 0 0.0000))
+    (property "Sheet name" "PowerSupply" (id 0) (at 27.94 24.6884 0)
+      (effects (font (size 1.27 1.27)) (justify left bottom))
+    )
+    (property "Sheet file" "Power-Supply.kicad_sch" (id 1) (at 27.94 69.1646 0)
       (effects (font (size 1.27 1.27)) (justify left top))
     )
@@
     (path "/" (page "1"))
     (path "/5942f19b-9c4c-4b0c-8e9c-1608ad5e1222" (page "2"))
+    (path "/a72be1e0-9af1-4c8b-a80a-e23a2ce6ded3" (page "3"))
   )
   (symbol_instances

Commit message: update the file
Other:
- sheet Audio Codec ports: added MCLK, SCL, SCLK, SDA, SDIN, SDOUT, ~{RST}; removed none

Commit message: update the file
Other:
- moved on the sheet: J5
Changed lines of the file:
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@@
     )
   )
-  (symbol (lib_id "1KiCadLib:SD-CARD-MEM2051-00-195-00-A") (at 229.87 119.38 0) (unit 1)
+  (symbol (lib_id "1KiCadLib:SD-CARD-MEM2051-00-195-00-A") (at 246.38 115.57 0) (unit 1)
     (in_bom yes) (on_board yes) (fields_autoplaced)
-    (property "Reference" "J5" (id 0) (at 229.87 104.14 0))
-    (property "Value" "SD-CARD-MEM2051-00-195-00-A" (id 1) (at 229.87 106.68 0))
-    (property "Footprint" "1KiCadLib:SD-CARD-MEM2051-00-195-00-A" (id 2) (at 227.33 104.14 0)
+    (property "Reference" "J5" (id 0) (at 246.38 100.33 0))
+    (property "Value" "SD-CARD-MEM2051-00-195-00-A" (id 1) (at 246.38 102.87 0))
+    (property "Footprint" "1KiCadLib:SD-CARD-MEM2051-00-195-00-A" (id 2) (at 243.84 100.33 0)
       (effects (font (size 1.27 1.27)) (justify bottom) hide)
     )
-    (property "Datasheet" "https://www.mouser.fr/ProductDetail/GCT/MEM2051-00-195-00-A?qs=KUoIvG%2F9Ilat7yfJRNWXUQ%3D%3D" (id 3) (at 229.87 105.41 0)
+    (property "Datasheet" "https://www.mouser.fr/ProductDetail/GCT/MEM2051-00-195-00-A?qs=KUoIvG%2F9Ilat7yfJRNWXUQ%3D%3D" (id 3) (at 246.38 101.6 0)
       (effects (font (size 1.27 1.27)) hide)
     )
-    (property "Manufacturer" "GCT" (id 4) (at 229.87 119.38 0)
+    (property "Manufacturer" "GCT" (id 4) (at 246.38 115.57 0)
       (effects (font (size 1.27 1.27)) (justify bottom) hide)
     )
-    (property "MPN" "MEM2051-00-195-00-A" (id 5) (at 226.06 97.79 0)
+    (property "MPN" "MEM2051-00-195-00-A" (id 5) (at 242.57 93.98 0)
       (effects (font (size 1.27 1.27)) hide)
     )
-    (property "Mouser" "640-MEM20510019500A" (id 6) (at 224.79 100.33 0)
+    (property "Mouser" "640-MEM20510019500A" (id 6) (at 241.3 96.52 0)
       (effects (font (size 1.27 1.27)) hide)
     )
@@
       (reference "#PWR0103") (unit 1) (value "GND") (footprint "")
     )
+    (path "/a72be1e0-9af1-4c8b-a80a-e23a2ce6ded3/2b097f79-705d-49b6-af61-336b3a0337f5"
+      (reference "#PWR?") (unit 1) (value "GND") (footprint "")
+    )
+    (path "/a72be1e0-9af1-4c8b-a80a-e23a2ce6ded3/37329a78-8994-4a1f-8c13-a0274929a527"
+      (reference "#PWR?") (unit 1) (value "GND") (footprint "")
+    )
+    (path "/a72be1e0-9af1-4c8b-a80a-e23a2ce6ded3/91e7bd5d-3ed4-494c-b6b0-e642be24bfd1"
+      (reference "#PWR?") (unit 1) (value "GND") (footprint "")
+    )
+    (path "/a72be1e0-9af1-4c8b-a80a-e23a2ce6ded3/cbc53a51-9b2d-4b0b-b990-0d5e86b29ced"
+      (reference "#PWR?") (unit 1) (value "GND") (footprint "")
+    )
+    (path "/a72be1e0-9af1-4c8b-a80a-e23a2ce6ded3/e502b510-7a0a-4ada-954f-66e05aed12cc"
+      (reference "#PWR?") (unit 1) (value "VBUS") (footprint "")
+    )
     (path "/5942f19b-9c4c-4b0c-8e9c-1608ad5e1222/263fa403-79b6-43fa-b2d9-5b6258649f66"
       (reference "C1") (unit 1) (value "22p") (footprint "Capacitor_SMD:C_0603_1608Metric")
@@
       (reference "C19") (unit 1) (value "100n") (footprint "Capacitor_SMD:C_0201_0603Metric")
     )
+    (path "/a72be1e0-9af1-4c8b-a80a-e23a2ce6ded3/6653ffe0-879a-46f2-b1d1-34b0ce318aaa"
+      (reference "C?") (unit 1) (value "10u") (footprint "Capacitor_SMD:C_0805_2012Metric")
+    )
+    (path "/a72be1e0-9af1-4c8b-a80a-e23a2ce6ded3/f4f41b56-17d1-47e1-9f78-609d3fae3725"
+      (reference "C?") (unit 1) (value "10u") (footprint "Capacitor_SMD:C_0805_2012Metric")
+    )
     (path "/147dd775-4cc4-4eb0-9062-db391a89cbc9"
       (reference "J1") (unit 1) (value "CON_USB_GCT_USB4105_REVA") (footprint "1KiCadLib:CON_USB_GCT_USB4105_REVA")
@@
       (reference "R10") (unit 1) (value "10K") (footprint "Resistor_SMD:R_0805_2012Metric")
     )
+    (path "/a72be1e0-9af1-4c8b-a80a-e23a2ce6ded3/4d24ff94-8066-4f90-93a1-a7d58b93e789"
+      (reference "R?") (unit 1) (value "2K") (footprint "Resistor_SMD:R_0805_2012Metric")
+    )
     (path "/5942f19b-9c4c-4b0c-8e9c-1608ad5e1222/0b60ea01-ae0f-4e02-bff3-d925c5e3ae76"
       (reference "U1") (unit 1) (value "CS42L51-CNZ") (footprint "Package_DFN_QFN:QFN-32-1EP_5x5mm_P0.5mm_EP3.1x3.1mm")
@@
       (reference "U2") (unit 1) (value "TLV73333PDBV") (footprint "Package_TO_SOT_SMD:SOT-23-5")
     )
-  )
+    (path "/a72be1e0-9af1-4c8b-a80a-e23a2ce6ded3/f70b8b80-e64f-4df8-8566-bb2d71d72144"
+      (reference "U?") (unit 1) (value "MCP73831-2-OT") (footprint "Package_TO_SOT_SMD:SOT-23-5")
+    )
+  )

Commit message: update the design
Parts:
- added C20: 4.7u, Capacitor_SMD:C_0805_2012Metric, symbol Device:C_Small
- added C21: 100n, Capacitor_SMD:C_0805_2012Metric, symbol Device:C_Small
- added C22, C23, C24, C26, C27, C28, C29, C30, C31, C32, C34, C35, C36, C38, C39, C40: 100n, Capacitor_SMD:C_0603_1608Metric, symbol Device:C_Small
- added C25, C33: 12p, Capacitor_SMD:C_0603_1608Metric, symbol Device:C_Small
- added C37: 2.2u, Capacitor_SMD:C_0603_1608Metric, symbol Device:C_Small
- added L1: 39n, symbol Device:L_Small
- added M4: MNT, MountingHole:MountingHole_2.1mm, symbol Mechanical:MountingHole
- added R11, R12, R13, R14, R15, R16, R17, R18: 10K, Resistor_SMD:R_0805_2012Metric, symbol Device:R_Small
- added SW1: RST, Button_Switch_SMD:SW_SPST_B3U-1000P-B, symbol Switch:SW_Push
- added U3: STM32H725ZET6, Package_QFP:LQFP-144_20x20mm_P0.5mm, symbol LibraryAudioBoard:STM32H725ZET6
- added Y1: 8MHz, symbol Device:Crystal_GND24
Connections:
- net GND: now also J5.6 (VSS), C20.2, C21.2, C22.2, C23.2, C24.2, C25.2, C26.2, C27.2, C28.2, C29.2, C30.2, C31.2, C32.2, C33.2, C34.2, C35.2, C36.2, C37.2, C38.2, C39.2, C40.2, R11.2, SW1.2, U3.104 (VSS), U3.118 (VSS), U3.12 (VSS), U3.128 (VSS), U3.14 (VSSSMPS), U3.141 (VSS), U3.18 (VSS), U3.33 (VSS), U3.34 (VSSA), U3.41 (VSS), U3.55 (VSS), U3.6 (VSS), U3.69 (VSS), U3.80 (VSS), U3.89 (VSS)
- net SD_D2: now reaches J5.1 (DATA2)
- net SD_D2: now also R16.2
- net SD_D3: now reaches J5.2 (DATA3/CD)
- net SD_D3: now also R15.2
- net SD_CMD: now reaches J5.3 (CMD)
- net SD_CMD: now also R14.2
- net +3.3V: now reaches J5.4 (VDD)
- net +3.3V: now also C22.1, C23.1, C24.1, C26.1, C27.1, C28.1, C30.1, C31.1, C32.1, C34.1, C36.1, C38.1, C39.1, C40.1, L1.2, R12.1, R13.1, R14.1, R15.1, R16.1, R17.1, R18.1, U3.105 (VDDLDO), U3.106 (VDD), U3.119 (VDD), U3.129 (VDD), U3.13 (VDD), U3.143 (VDDLDO), U3.144 (VDD), U3.19 (VDD), U3.32 (VDD), U3.42 (VDD), U3.56 (VDD), U3.7 (VDD), U3.70 (VDDLDO), U3.71 (VDD), U3.79 (VDD), U3.8 (VBAT), U3.91 (VDD33USB), U3.92 (VDD)
- net SD_CLK: now reaches J5.5 (CLK)
- net SD_D0: now reaches J5.7 (DATA0)
- net SD_D0: now also R18.2
- net SD_D1: now reaches J5.8 (DATA1)
- net SD_D1: now also R17.2
- new net: C35.1, C37.1, L1.1, U3.35 (VREF+), U3.36 (VDDA)
- new net: C29.1, R13.2, SW1.1, U3.27 (NRST)
- new net: C33.1, U3.26 (PH1-OSC_OUT), Y1.3
- new net: C25.1, U3.25 (PH0-OSC_IN), Y1.1
- new net: R12.2, U3.142 (PDR_ON)
- new net: C20.1, C21.1, U3.103 (VCAP), U3.140 (VCAP), U3.68 (VCAP)
- new net: R11.1, U3.135 (BOOT0)
- new net: Y1.2, Y1.4
- no-connect marks 0 -> 3
Other:
- note added: "STM32H725ZET6"
- moved on the sheet: J1, J5, M1, M2, M3

Commit message: update the design
Parts:
- removed C20: 4.7u, Capacitor_SMD:C_0805_2012Metric, symbol Device:C_Small
- removed C21: 100n, Capacitor_SMD:C_0805_2012Metric, symbol Device:C_Small
- removed C22, C23, C24, C26, C27, C28, C29, C30, C31, C32, C34, C35, C36, C38, C39: 100n, Capacitor_SMD:C_0603_1608Metric, symbol Device:C_Small
- removed C25, C33: 12p, Capacitor_SMD:C_0603_1608Metric, symbol Device:C_Small
- removed C37: 2.2u, Capacitor_SMD:C_0603_1608Metric, symbol Device:C_Small
- removed L1: 39n, symbol Device:L_Small
- removed R11, R12, R13: 10K, Resistor_SMD:R_0805_2012Metric, symbol Device:R_Small
- removed SW1: RST, Button_Switch_SMD:SW_SPST_B3U-1000P-B, symbol Switch:SW_Push
- removed U3: STM32H725ZET6, Package_QFP:LQFP-144_20x20mm_P0.5mm, symbol LibraryAudioBoard:STM32H725ZET6
- removed Y1: 8MHz, symbol Device:Crystal_GND24
- added C?: 100n, Capacitor_SMD:C_0603_1608Metric, symbol Device:C_Small
- added C?: 4.7u, Capacitor_SMD:C_0805_2012Metric, symbol Device:C_Small
- added C? (x2): 12p, Capacitor_SMD:C_0603_1608Metric, symbol Device:C_Small
- added J?: STLINK, Connector_PinHeader_2.54mm:PinHeader_1x04_P2.54mm_Vertical, symbol Connector_Generic:Conn_01x04
- added R? (x2): 10K, Resistor_SMD:R_0805_2012Metric, symbol Device:R_Small
- added SW?: RST, Button_Switch_SMD:SW_SPST_B3U-1000P-B, symbol Switch:SW_Push
- added U?: STM32F446RETx, Package_QFP:LQFP-64_10x10mm_P0.5mm, symbol MCU_ST_STM32F4:STM32F446RETx
- added Y?: 8MHz, Crystal:Crystal_SMD_3225-4Pin_3.2x2.5mm, symbol Device:Crystal_GND24
Connections:
- net +3.3V: now also J?.1 (Pin_1), R?.1, U?.1 (VBAT), U?.13 (VDDA), U?.19 (VDD), U?.32 (VDD), U?.48 (VDD), U?.64 (VDD)
- net GND: now also C?.2, C?.2, C?.2, C?.2, J?.4 (Pin_4), R?.1, SW?.2, U?.12 (VSSA), U?.18 (VSS), U?.31 (VSS), U?.47 (VSS), U?.63 (VSS)
- net SD_CLK renamed SD_CLK_PB2
- net SD_CMD renamed SD_CMD_PD2
- net SD_D0 renamed SD_D0_PC8
- net SD_D1 renamed SD_D1_PB0
- net SD_D2 renamed SD_D2_PB1
- net SD_D3 renamed SD_D3_PC11
- new net: C?.1, R?.2, SW?.1, U?.7 (NRST)
- new net: R?.2, U?.60 (BOOT0)
- new net: C?.1, U?.30 (VCAP_1)
- new net: Y?.2, Y?.4
- new net SWCLK_PA14: J?.2 (Pin_2), U?.49 (PA14)
- new net SWDIO_PA13: J?.3 (Pin_3), U?.50 (PA15)
- new net XIN: C?.1, U?.5 (PH0), Y?.1
- new net XOUT: C?.1, U?.6 (PH1), Y?.3
- no-connect marks 3 -> 0
Other:
- added sheet STM32H7 (STM32H7.kicad_sch)
- note removed: "STM32H725ZET6"
- moved on the sheet: C40, J1, J5, R14, R15, R16, R17, R18

Commit message: update the design
Parts:
- added U?: D-ESD-PESD2ETH-AD, Package_TO_SOT_SMD:SOT-23-6, symbol 1KiCadLib:D-ESD-PESD2ETH-AD
Connections:
- net GND: now also U?.2 (GND)
- net SD_CLK_PB2: now also U?.28 (PB2)
- net SD_CMD_PD2: now also U?.54 (PD2)
- net SD_D0_PC8: now also U?.39 (PC8)
- net SD_D1_PB0: now also U?.26 (PB0)
- net SD_D2_PB1: now also U?.27 (PB1)
- net SD_D3_PC11: now also U?.52 (PC11)
- net USB_POWER: now reaches J1.A4/B9 (VBUS), J1.B4/A9 (VBUS)
- net USB_POWER: now also U?.5 (VBUS)
- net USB+: now reaches J1.A6 (DP1)
- net USB+: now also J1.B6 (DP2), U?.6 (I/O1)
- net USB-: now reaches J1.A7 (DN1)
- net USB-: now also J1.B7 (DN2), U?.4 (I/O2)
- net USB_N: now reaches U?.44 (PA11)
- net USB_N: now also U?.3 (I/O2)
- net USB_P: now reaches U?.45 (PA12)
- net USB_P: now also U?.1 (I/O1)
- no-connect marks 0 -> 2
Other:
- note added: "SD Card With SDIO Interface"
- note added: "USB HOST Interface"
- moved on the sheet: C40, J1, J5, R14, R15, R16, R17, R18
