File: hardware/AUDIO-BOARD.kicad_sch (KiCad schematic)
At the start: 23 parts, among them J1 CON_USB_GCT_USB4105_REVA, J5 SD-CARD-MEM2051-00-195-00-A, M1 MNT, M2 MNT, M3 MNT, M4 MNT

Commit message: update the design
Other:
- sheet Audio Codec ports: added LRCK; removed none
Changed lines of the file:
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@@
   (no_connect (at 41.91 148.59))
   (no_connect (at 41.91 151.13))
-  (wire (pts (xy 125.73 106.68) (xy 128.27 106.68))
+  (wire (pts (xy 125.73 101.6) (xy 128.27 101.6))
     (stroke (width 0) (type default) (color 0 0 0 0))
   )
@@
     (stroke (width 0) (type default) (color 0 0 0 0))
   )
-  (wire (pts (xy 125.73 99.06) (xy 128.27 99.06))
+  (wire (pts (xy 125.73 93.98) (xy 128.27 93.98))
     (stroke (width 0) (type default) (color 0 0 0 0))
   )
@@
     (stroke (width 0) (type default) (color 0 0 0 0))
   )
+  (wire (pts (xy 125.73 109.22) (xy 128.27 109.22))
+    (stroke (width 0) (type default) (color 0 0 0 0))
+  )
   (wire (pts (xy 205.74 25.4) (xy 205.74 22.86))
     (stroke (width 0) (type default) (color 0 0 0 0))
@@
     (stroke (width 0) (type default) (color 0 0 0 0))
   )
-  (wire (pts (xy 125.73 102.87) (xy 128.27 102.87))
+  (wire (pts (xy 125.73 97.79) (xy 128.27 97.79))
     (stroke (width 0) (type default) (color 0 0 0 0))
   )
@@
     (stroke (width 0) (type default) (color 0 0 0 0))
   )
+  (wire (pts (xy 125.73 116.84) (xy 128.27 116.84))
+    (stroke (width 0) (type default) (color 0 0 0 0))
+  )
   (wire (pts (xy 27.94 58.42) (xy 24.13 58.42))
     (stroke (width 0) (type default) (color 0 0 0 0))
@@
     (stroke (width 0) (type default) (color 0 0 0 0))
   )
-  (wire (pts (xy 125.73 110.49) (xy 128.27 110.49))
+  (wire (pts (xy 125.73 105.41) (xy 128.27 105.41))
     (stroke (width 0) (type default) (color 0 0 0 0))
   )
@@
   )
   (wire (pts (xy 41.91 35.56) (xy 48.26 35.56))
+    (stroke (width 0) (type default) (color 0 0 0 0))
+  )
+  (wire (pts (xy 125.73 113.03) (xy 128.27 113.03))
     (stroke (width 0) (type default) (color 0 0 0 0))
   )
@@
     )
   )
+  (global_label "I2C_SDA_PB7" (shape input) (at 125.73 116.84 180) (fields_autoplaced)
+    (effects (font (size 1 1)) (justify right))
+    (property "Intersheet References" "${INTERSHEET_REFS}" (id 0) (at 114.1157 116.7775 0)
+      (effects (font (size 1 1)) (justify right) hide)
+    )
+  )
   (global_label "SD_CLK_PB2" (shape bidirectional) (at 99.06 78.74 0) (fields_autoplaced)
     (effects (font (size 1 1)) (justify left))
@@
     )
   )
-  (global_label "I2S_SCLK_PA5" (shape input) (at 125.73 102.87 180) (fields_autoplaced)
-    (effects (font (size 1 1)) (justify right))
-    (property "Intersheet References" "${INTERSHEET_REFS}" (id 0) (at 113.3538 102.8075 0)
+  (global_label "I2S_SCLK_PA5" (shape input) (at 125.73 97.79 180) (fields_autoplaced)
+    (effects (font (size 1 1)) (justify right))
+    (property "Intersheet References" "${INTERSHEET_REFS}" (id 0) (at 113.3538 97.7275 0)
       (effects (font (size 1 1)) (justify right) hide)
     )
@@
     )
   )
+  (global_label "I2S_WS_PA4" (shape input) (at 125.73 109.22 180) (fields_autoplaced)
+    (effects (font (size 1 1)) (justify right))
+    (property "Intersheet References" "${INTERSHEET_REFS}" (id 0) (at 115.0205 109.1575 0)
+      (effects (font (size 1 1)) (justify right) hide)
+    )
+  )
   (global_label "USB-" (shape output) (at 49.53 160.02 0) (fields_autoplaced)
     (effects (font (size 1 1)) (justify left))
@@
     )
   )
-  (global_label "I2S_DIN_PA7" (shape input) (at 125.73 110.49 180) (fields_autoplaced)
-    (effects (font (size 1 1)) (justify right))
-    (property "Intersheet References" "${INTERSHEET_REFS}" (id 0) (at 114.5919 110.4275 0)
-      (effects (font (size 1 1)) (justify right) hide)
-    )
-  )
-  (global_label "I2S_DOUT" (shape output) (at 125.73 99.06 180) (fields_autoplaced)
-    (effects (font (size 1 1)) (justify right))
-    (property "Intersheet References" "${INTERSHEET_REFS}" (id 0) (at 116.83 98.9975 0)
+  (global_label "I2C_SCL_PB6" (shape input) (at 125.73 113.03 180) (fields_autoplaced)
+    (effects (font (size 1 1)) (justify right))
+    (property "Intersheet References" "${INTERSHEET_REFS}" (id 0) (at 114.1633 112.9675 0)
+      (effects (font (size 1 1)) (justify right) hide)
+    )
+  )
+  (global_label "I2S_DIN_PA7" (shape input) (at 125.73 105.41 180) (fields_autoplaced)
+    (effects (font (size 1 1)) (justify right))
+    (property "Intersheet References" "${INTERSHEET_REFS}" (id 0) (at 114.5919 105.3475 0)
+      (effects (font (size 1 1)) (justify right) hide)
+    )
+  )
+  (global_label "I2S_DOUT" (shape output) (at 125.73 93.98 180) (fields_autoplaced)
+    (effects (font (size 1 1)) (justify right))
+    (property "Intersheet References" "${INTERSHEET_REFS}" (id 0) (at 116.83 93.9175 0)
       (effects (font (size 1 1)) (justify right) hide)
     )
@@
     )
   )
-  (global_label "I2S_MCLK_PC4" (shape input) (at 125.73 106.68 180) (fields_autoplaced)
-    (effects (font (size 1 1)) (justify right))
-    (property "Intersheet References" "${INTERSHEET_REFS}" (id 0) (at 113.0205 106.6175 0)
+  (global_label "I2S_MCLK_PC4" (shape input) (at 125.73 101.6 180) (fields_autoplaced)
+    (effects (font (size 1 1)) (justify right))
+    (property "Intersheet References" "${INTERSHEET_REFS}" (id 0) (at 113.0205 101.5375 0)
       (effects (font (size 1 1)) (justify right) hide)
     )
@@
     )
   )
-  (sheet (at 128.27 93.98) (size 27.94 27.94) (fields_autoplaced)
+  (sheet (at 128.27 88.9) (size 27.94 30.48) (fields_autoplaced)
     (stroke (width 0.1524) (type solid) (color 128 77 0 1))
     (fill (color 255 255 194 1.0000))
-    (property "Sheet name" "Audio Codec" (id 0) (at 128.27 93.2684 0)
+    (property "Sheet name" "Audio Codec" (id 0) (at 128.27 88.1884 0)
       (effects (font (size 1.27 1.27)) (justify left bottom))
     )
-    (property "Sheet file" "audio-codec.kicad_sch" (id 1) (at 128.27 122.5046 0)
+    (property "Sheet file" "audio-codec.kicad_sch" (id 1) (at 128.27 119.9646 0)
       (effects (font (size 1.27 1.27)) (justify left top))
     )
-    (pin "~{RST}" input (at 128.27 95.25 180)
-      (effects (font (size 1.27 1.27)) (justify left))
-    )
-    (pin "SCL" input (at 128.27 114.3 180)
-      (effects (font (size 1.27 1.27)) (justify left))
-    )
-    (pin "SDOUT" output (at 128.27 99.06 180)
-      (effects (font (size 1.27 1.27)) (justify left))
-    )
-    (pin "SCLK" input (at 128.27 102.87 180)
-      (effects (font (size 1.27 1.27)) (justify left))
-    )
-    (pin "MCLK" input (at 128.27 106.68 180)
-      (effects (font (size 1.27 1.27)) (justify left))
-    )
-    (pin "SDIN" input (at 128.27 110.49 180)
-      (effects (font (size 1.27 1.27)) (justify left))
-    )
-    (pin "SDA" bidirectional (at 128.27 118.11 180)
-      (effects (font (size 1.27 1.27)) (justify left))
-    )
+    (pin "~{RST}" input (at 128.27 90.17 180)
+      (effects (font (size 1.27 1.27)) (justify left))
+    )
+    (pin "SCL" input (at 128.27 113.03 180)
+      (effects (font (size 1.27 1.27)) (justify left))
+    )
+    (pin "SDOUT" output (at 128.27 93.98 180)
+      (effects (font (size 1.27 1.27)) (justify left))
+    )
+    (pin "SCLK" input (at 128.27 97.79 180)
+      (effects (font (size 1.27 1.27)) (justify left))
+    )
+    (pin "MCLK" input (at 128.27 101.6 180)
+      (effects (font (size 1.27 1.27)) (justify left))
+    )
+    (pin "SDIN" input (at 128.27 105.41 180)
+      (effects (font (size 1.27 1.27)) (justify left))
+    )
+    (pin "SDA" bidirectional (at 128.27 116.84 180)
+      (effects (font (size 1.27 1.27)) (justify left))
+    )
+    (pin "LRCK" input (at 128.27 109.22 180)
+      (effects (font (size 1.27 1.27)) (justify left))
+    )

Commit message: update the design
Parts:
- added C? (x6): 100n, Capacitor_SMD:C_0603_1608Metric, symbol Device:C_Small
Connections:
- net +3.3V: now also C?.1, C?.1, C?.1, C?.1, C?.1, C?.1
- net GND: now also C?.2, C?.2, C?.2, C?.2, C?.2, C?.2
Other:
- sheet Audio Codec ports: added M/~{S}; removed SDOUT
- moved on the sheet: J?

Commit message: update the design
Parts:
- added C?: 100n, Capacitor_SMD:C_0603_1608Metric, symbol Device:C_Small
- added R4, R6: 10K, Resistor_SMD:R_0805_2012Metric, symbol Device:R_Small
- added U?: TSOP38G36, OptoDevice:Vishay_MINICAST-3Pin, symbol Interface_Optical:TSOP38G36
- gave numbers to parts that had none: 17
- renumbered C40 to C11, J5 to J3, R14 to R3, R15 to R5, R16 to R7, R17 to R8, R18 to R9
Connections:
- net +3.3V: now also C?.1, R4.1, R6.1, U?.3 (Vs)
- net GND: now also C?.2, U?.2 (GND)
- net I2C_SCL_PB6: now also U1.58 (PB6), R6.2
- net I2C_SDA_PB7: now also U1.59 (PB7), R4.2
- net I2S_DIN_PA7: now also U1.23 (PA7)
- net I2S_MCLK_PC4: now also U1.24 (PC4)
- net I2S_SCLK_PA5: now also U1.21 (PA5)
- net I2S_WS_PA4: now also U1.20 (PA4)
- new net IRR_OUT: U?.1 (OUT)
Other:
- removed sheet STM32H7
- note added: "38kHz"
- note added: "Infra Red Receicer Interface"

Commit message: update the design
Parts:
- gave numbers to parts that had none: 2
- renumbered C11 to C12

Commit message: update the design
Parts:
- added D1: LED, LED_SMD:LED_0805_2012Metric, symbol Device:LED
- added R16: 1K, Resistor_SMD:R_0805_2012Metric, symbol Device:R_Small
Connections:
- net +3.3V: now also R16.1
- net GND: now also D1.1 (K)
- new net: D1.2 (A), R16.2
Other:
- sheet PowerSupply ports: added USB_OTG_EN, USB_OTG_VBUS; removed none
- note added: "Audio Codec Interface"
- note added: "Power Supplies"
- moved on the sheet: C1, C10, C11, C12, C2, C3, C4, C5, C6, C7, C8, C9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

Commit message: Update placements
Connections:
- net GND: now also J3.10 (SHIELD)
- net IRR_OUT: now also U1.36 (PB15)
- net USB_OTG_EN: now also U1.33 (PB12)
- no-connect marks 2 -> 3
Other:
- moved on the sheet: C12, J2

Commit message: Update the PCB routing
Parts:
- added J8: TFT TOUCH SCREEN, Connector_PinSocket_2.54mm:PinSocket_1x14_P2.54mm_Vertical, symbol Connector_Generic:Conn_01x14
Connections:
- net USB_POWER is gone; now on net USB_OTG_VBUS: J1.A4/B9 (VBUS), J1.B4/A9 (VBUS), U2.5 (VBUS)
- net +3.3V: now also J8.1 (Pin_1)
- net GND: now also J8.2 (Pin_2)
- net SPI2_MISO_PC2: now reaches U1.10 (PC2)
- net SPI2_MISO_PC2: now also J8.9 (Pin_9)
- net SPI3_nCS_PC13: now reaches U1.2 (PC13)
- net SPI3_nCS_PC13: now also J8.11 (Pin_11)
- net SPI2_SCK_PB10: now reaches U1.29 (PB10)
- net SPI2_SCK_PB10: now also J8.7 (Pin_7)
- net LCD_RST_PC14: now reaches U1.3 (PC14)
- net LCD_RST_PC14: now also J8.4 (Pin_4)
- net LCD_LED_PC6: now reaches U1.37 (PC6)
- net LCD_LED_PC6: now also J8.8 (Pin_8)
- net LCD_T_IRQ_PC7: now reaches U1.38 (PC7)
- net LCD_T_IRQ_PC7: now also J8.14 (Pin_14)
- net LCD_DC_PC15: now reaches U1.4 (PC15)
- net LCD_DC_PC15: now also J8.5 (Pin_5)
- net SPI3_SCK_PC10: now reaches U1.51 (PC10)
- net SPI3_SCK_PC10: now also J8.10 (Pin_10)
- net SPI3_MOSI_PC12: now reaches U1.53 (PC12)
- net SPI3_MOSI_PC12: now also J8.12 (Pin_12)
- net SPI3_MISO_PB4: now reaches U1.56 (PB4)
- net SPI3_MISO_PB4: now also J8.13 (Pin_13)
- net SPI2_nCS_PB9: now reaches U1.62 (PB9)
- net SPI2_nCS_PB9: now also J8.3 (Pin_3)
- net SPI2_MOSI_PC1: now reaches U1.9 (PC1)
- net SPI2_MOSI_PC1: now also J8.6 (Pin_6)
- no-connect marks 3 -> 5
Other:
- moved on the sheet: C1, C3, C4, D1, R16, U2, Y1
