File: hardware/Power-Supply.kicad_sch (KiCad schematic)
At the start: 0 parts

Commit message: Updating the power section
Parts:
- added C? (x2): 10u, Capacitor_SMD:C_0805_2012Metric, symbol Device:C_Small
- added C?: 100n, Capacitor_SMD:C_0201_0603Metric, symbol Device:C_Small
- added J?: BATT, Connector_JST:JST_EH_S2B-EH_1x02_P2.50mm_Horizontal, symbol Connector_Generic:Conn_01x02
- added J?: CON_USB_GCT_USB4105_REVA, 1KiCadLib:CON_USB_GCT_USB4105_REVA, symbol 1KiCadLib:CON_USB_GCT_USB4105_REVA
- added Q? (x4): DMP3013SFV-7, CM4IO:Diodes_PowerDI3333-8, symbol Transistor_FET:DMP3013SFV
- added Q? (x2): SI2324DS-T1-GE3, Package_TO_SOT_SMD:SOT-23, symbol Device:Q_NMOS_GSD
- added R? (x2): 10K, Resistor_SMD:R_0805_2012Metric, symbol Device:R_Small
- added R? (x3): 100K, Resistor_SMD:R_0805_2012Metric, symbol Device:R_Small
- added R?: 330R, Resistor_SMD:R_0805_2012Metric, symbol Device:R_Small
- added U?: TLV73333PDBV, Package_TO_SOT_SMD:SOT-23-5, symbol Regulator_Linear:TLV73333PDBV
Connections:
- new net: C?.1, U?.1 (IN)
- new net: Q?.1 (S), Q?.2 (S), Q?.3 (S), Q?.5 (D), R?.1 (x2)
- new net: Q?.3 (D), Q?.4 (G), Q?.4 (G), R?.2, R?.2
- new net: C?.1, Q?.1 (G), R?.1, R?.2
- new net: Q?.1 (G), R?.1, R?.2
- new net: Q?.3 (D), Q?.4 (G), Q?.4 (G), R?.2
- new net +3.3V: C?.1, U?.5 (OUT)
- new net +BATT: J?.2 (Pin_2)
- new net +VBAT: Q?.5 (D), R?.1
- new net DC_INPUT_OR_+VBAT: Q?.1 (S), Q?.1 (S), Q?.2 (S), Q?.2 (S), Q?.3 (S), Q?.3 (S)
- new net GND: C?.2, C?.2, C?.2, J?.1 (Pin_1), J?.A1/B12 (GND), J?.B1/A12 (GND), J?.G1 (GND), J?.G2 (GND), J?.G3 (GND), J?.G4 (GND), Q?.2 (S), Q?.2 (S), R?.2, U?.2 (GND)
- new net VBUS: J?.A4/B9 (VBUS), J?.B4/A9 (VBUS)
- new net VUSB: Q?.5 (D), R?.1
- no-connect marks 0 -> 2
Other:
- note added: "Power input selection (DC input or Battery Input)"
- note added: "TJ15P04M3,RQ(S"
- note added: "The priority is given to the +5V DC input. When the DC input voltage is presen, the battery source is not used ."

Commit message: update the file
Connections:
- net at C?.1, U?.1 (IN): now also U?.3 (EN)
Changed lines of the file:
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@@
   (junction (at 76.2 81.28) (diameter 0) (color 0 0 0 0)
+  )
+  (junction (at 223.52 27.94) (diameter 0) (color 0 0 0 0)
   )
   (junction (at 77.47 31.75) (diameter 0) (color 0 0 0 0)
@@
   )
   (wire (pts (xy 77.47 62.23) (xy 77.47 69.85))
+    (stroke (width 0) (type default) (color 0 0 0 0))
+  )
+  (wire (pts (xy 227.33 30.48) (xy 223.52 30.48))
     (stroke (width 0) (type default) (color 0 0 0 0))
   )
@@
     (stroke (width 0) (type default) (color 0 0 0 0))
   )
+  (wire (pts (xy 223.52 27.94) (xy 217.17 27.94))
+    (stroke (width 0) (type default) (color 0 0 0 0))
+  )
   (wire (pts (xy 68.58 31.75) (xy 77.47 31.75))
     (stroke (width 0) (type default) (color 0 0 0 0))
@@
   )
   (wire (pts (xy 217.17 27.94) (xy 217.17 29.21))
+    (stroke (width 0) (type default) (color 0 0 0 0))
+  )
+  (wire (pts (xy 223.52 30.48) (xy 223.52 27.94))
     (stroke (width 0) (type default) (color 0 0 0 0))
   )
@@
     (stroke (width 0) (type default) (color 0 0 0 0))
   )
-  (wire (pts (xy 227.33 27.94) (xy 217.17 27.94))
+  (wire (pts (xy 227.33 27.94) (xy 223.52 27.94))
     (stroke (width 0) (type default) (color 0 0 0 0))
   )

Commit message: update the file
Parts:
- removed C?: 100n, Capacitor_SMD:C_0201_0603Metric, symbol Device:C_Small
- removed Q? (x4): DMP3013SFV-7, CM4IO:Diodes_PowerDI3333-8, symbol Transistor_FET:DMP3013SFV
- removed Q? (x2): SI2324DS-T1-GE3, Package_TO_SOT_SMD:SOT-23, symbol Device:Q_NMOS_GSD
- removed R? (x2): 10K, Resistor_SMD:R_0805_2012Metric, symbol Device:R_Small
- removed R? (x3): 100K, Resistor_SMD:R_0805_2012Metric, symbol Device:R_Small
- removed R?: 330R, Resistor_SMD:R_0805_2012Metric, symbol Device:R_Small
- gave numbers to parts that had none: 5
Connections:
- net DC_OUT: now reaches C17.1, U2.1 (IN), U2.3 (EN)
Other:
- added sheet PowerSelector (PowerSelector.kicad_sch)
- note removed: "Power input selection (DC input or Battery Input)"
- note removed: "TJ15P04M3,RQ(S"
- note removed: "The priority is given to the +5V DC input. When the DC input voltage is presen, the battery source is not used ."
- moved on the sheet: C17, C18, J3, J4, U2

Commit message: update the file
Parts:
- added C? (x2): 10u, Capacitor_SMD:C_0805_2012Metric, symbol Device:C_Small
- added R?: 2K, Resistor_SMD:R_0805_2012Metric, symbol Device:R_Small
- added U?: MCP73831-2-OT, Package_TO_SOT_SMD:SOT-23-5, symbol Battery_Management:MCP73831-2-OT
Connections:
- net +BATT: now also C?.1, U?.3 (VBAT)
- net GND: now also C?.2, C?.2, R?.2, U?.2 (VSS)
- net VBUS: now also C?.1, U?.4 (VDD)
- new net: R?.1, U?.5 (PROG)
Other:
- moved on the sheet: C17, C18, J4, U2

Commit message: update the design
Parts:
- gave numbers to parts that had none: 4
Changed lines of the file:
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@@
   (symbol (lib_id "power:GND") (at 124.46 105.41 0) (unit 1)
     (in_bom yes) (on_board yes) (fields_autoplaced)
-    (property "Reference" "#PWR?" (id 0) (at 124.46 111.76 0)
+    (property "Reference" "#PWR052" (id 0) (at 124.46 111.76 0)
       (effects (font (size 1.27 1.27)) hide)
     )
@@
   (symbol (lib_id "power:GND") (at 148.59 104.14 0) (unit 1)
     (in_bom yes) (on_board yes) (fields_autoplaced)
-    (property "Reference" "#PWR?" (id 0) (at 148.59 110.49 0)
+    (property "Reference" "#PWR053" (id 0) (at 148.59 110.49 0)
       (effects (font (size 1.27 1.27)) hide)
     )
@@
   (symbol (lib_id "Device:R_Small") (at 113.03 101.6 0) (unit 1)
     (in_bom yes) (on_board yes) (fields_autoplaced)
-    (property "Reference" "R?" (id 0) (at 115.57 100.3299 0)
+    (property "Reference" "R19" (id 0) (at 115.57 100.3299 0)
       (effects (font (size 1.27 1.27)) (justify left))
     )
@@
   (symbol (lib_id "Device:C_Small") (at 105.41 96.52 0) (unit 1)
     (in_bom yes) (on_board yes) (fields_autoplaced)
-    (property "Reference" "C?" (id 0) (at 107.95 95.2562 0)
+    (property "Reference" "C41" (id 0) (at 107.95 95.2562 0)
       (effects (font (size 1.27 1.27)) (justify left))
     )
@@
   (symbol (lib_id "power:GND") (at 113.03 105.41 0) (unit 1)
     (in_bom yes) (on_board yes) (fields_autoplaced)
-    (property "Reference" "#PWR?" (id 0) (at 113.03 111.76 0)
+    (property "Reference" "#PWR050" (id 0) (at 113.03 111.76 0)
       (effects (font (size 1.27 1.27)) hide)
     )
@@
   (symbol (lib_id "power:GND") (at 105.41 105.41 0) (unit 1)
     (in_bom yes) (on_board yes) (fields_autoplaced)
-    (property "Reference" "#PWR?" (id 0) (at 105.41 111.76 0)
+    (property "Reference" "#PWR049" (id 0) (at 105.41 111.76 0)
       (effects (font (size 1.27 1.27)) hide)
     )
@@
   (symbol (lib_id "power:VBUS") (at 124.46 83.82 0) (unit 1)
     (in_bom yes) (on_board yes)
-    (property "Reference" "#PWR?" (id 0) (at 124.46 87.63 0)
+    (property "Reference" "#PWR051" (id 0) (at 124.46 87.63 0)
       (effects (font (size 1.27 1.27)) hide)
     )
@@
   (symbol (lib_id "Device:C_Small") (at 148.59 96.52 0) (unit 1)
     (in_bom yes) (on_board yes) (fields_autoplaced)
-    (property "Reference" "C?" (id 0) (at 151.13 95.2562 0)
+    (property "Reference" "C42" (id 0) (at 151.13 95.2562 0)
       (effects (font (size 1.27 1.27)) (justify left))
     )
@@
   (symbol (lib_id "Battery_Management:MCP73831-2-OT") (at 124.46 93.98 0) (unit 1)
     (in_bom yes) (on_board yes) (fields_autoplaced)
-    (property "Reference" "U?" (id 0) (at 126.4794 83.82 0)
-      (effects (font (size 1.27 1.27)) (justify left))
-    )
+    (property "Reference" "U4" (id 0) (at 126.4794 83.82 0)
+      (effects (font (size 1.27 1.27)) (justify left))
+    )

Commit message: update the design
Parts:
- added C? (x2): 10u, Capacitor_SMD:C_0805_2012Metric, symbol Device:C_Small
- added U?: NCP163ASN280T1G, Package_TO_SOT_SMD:SOT-23-5, symbol Regulator_Linear:NCP163ASN280T1G
Connections:
- net DC_OUT: now also C?.1, U?.1 (VIN), U?.3 (EN)
- net GND: now also C?.2, C?.2, U?.2 (GND)
- new net +2V5: C?.1, U?.5 (VOUT)
Other:
- note added: "3V3 Regulator for the Audio Codec @250mA"
- note added: "3V3 Regulator for the MCU @300mA"
Changed lines of the file:
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@@
   (junction (at 254 33.02) (diameter 0) (color 0 0 0 0)
+  )
+  (junction (at 223.52 91.44) (diameter 0) (color 0 0 0 0)
+  )
+  (junction (at 229.87 91.44) (diameter 0) (color 0 0 0 0)
+  )
+  (junction (at 254 91.44) (diameter 0) (color 0 0 0 0)
   )
   (junction (at 223.52 33.02) (diameter 0) (color 0 0 0 0)
@@
     (stroke (width 0) (type default) (color 0 0 0 0))
   )
+  (wire (pts (xy 229.87 96.52) (xy 229.87 91.44))
+    (stroke (width 0) (type default) (color 0 0 0 0))
+  )
   (wire (pts (xy 148.59 99.06) (xy 148.59 104.14))
     (stroke (width 0) (type default) (color 0 0 0 0))
@@
     (stroke (width 0) (type default) (color 0 0 0 0))
   )
+  (wire (pts (xy 233.68 91.44) (xy 229.87 91.44))
+    (stroke (width 0) (type default) (color 0 0 0 0))
+  )
   (wire (pts (xy 233.68 35.56) (xy 229.87 35.56))
     (stroke (width 0) (type default) (color 0 0 0 0))
@@
     (stroke (width 0) (type default) (color 0 0 0 0))
   )
+  (polyline (pts (xy 283.21 72.39) (xy 193.04 72.39))
+    (stroke (width 0) (type default) (color 0 0 0 0))
+  )
+  (wire (pts (xy 215.9 91.44) (xy 223.52 91.44))
+    (stroke (width 0) (type default) (color 0 0 0 0))
+  )
+  (wire (pts (xy 254 97.79) (xy 254 104.14))
+    (stroke (width 0) (type default) (color 0 0 0 0))
+  )
   (polyline (pts (xy 13.97 133.35) (xy 13.97 72.39))
     (stroke (width 0) (type default) (color 0 0 0 0))
   )
+  (polyline (pts (xy 193.04 72.39) (xy 193.04 133.35))
+    (stroke (width 0) (type default) (color 0 0 0 0))
+  )
+  (wire (pts (xy 233.68 96.52) (xy 229.87 96.52))
+    (stroke (width 0) (type default) (color 0 0 0 0))
+  )
   (wire (pts (xy 113.03 104.14) (xy 113.03 105.41))
     (stroke (width 0) (type default) (color 0 0 0 0))
@@
     (stroke (width 0) (type default) (color 0 0 0 0))
   )
+  (polyline (pts (xy 193.04 133.35) (xy 283.21 133.35))
+    (stroke (width 0) (type default) (color 0 0 0 0))
+  )
   (wire (pts (xy 158.75 91.44) (xy 158.75 90.17))
     (stroke (width 0) (type default) (color 0 0 0 0))
@@
     (stroke (width 0) (type default) (color 0 0 0 0))
   )
+  (wire (pts (xy 223.52 91.44) (xy 223.52 92.71))
+    (stroke (width 0) (type default) (color 0 0 0 0))
+  )
   (wire (pts (xy 254 39.37) (xy 254 45.72))
     (stroke (width 0) (type default) (color 0 0 0 0))
@@
     (stroke (width 0) (type default) (color 0 0 0 0))
   )
+  (wire (pts (xy 254 92.71) (xy 254 91.44))
+    (stroke (width 0) (type default) (color 0 0 0 0))
+  )
   (wire (pts (xy 158.75 95.25) (xy 158.75 91.44))
     (stroke (width 0) (type default) (color 0 0 0 0))
@@
     (stroke (width 0) (type default) (color 0 0 0 0))
   )
+  (wire (pts (xy 254 91.44) (xy 248.92 91.44))
+    (stroke (width 0) (type default) (color 0 0 0 0))
+  )
   (wire (pts (xy 124.46 85.09) (xy 124.46 86.36))
     (stroke (width 0) (type default) (color 0 0 0 0))
@@
     (stroke (width 0) (type default) (color 0 0 0 0))
   )
+  (wire (pts (xy 223.52 97.79) (xy 223.52 104.14))
+    (stroke (width 0) (type default) (color 0 0 0 0))
+  )
   (wire (pts (xy 148.59 93.98) (xy 148.59 91.44))
     (stroke (width 0) (type default) (color 0 0 0 0))
@@
     (stroke (width 0) (type default) (color 0 0 0 0))
   )
+  (polyline (pts (xy 283.21 133.35) (xy 283.21 72.39))
+    (stroke (width 0) (type default) (color 0 0 0 0))
+  )
   (wire (pts (xy 105.41 99.06) (xy 105.41 105.41))
     (stroke (width 0) (type default) (color 0 0 0 0))
@@
     (stroke (width 0) (type default) (color 0 0 0 0))
   )
+  (wire (pts (xy 241.3 101.6) (xy 241.3 104.14))
+    (stroke (width 0) (type default) (color 0 0 0 0))
+  )
   (polyline (pts (xy 90.17 72.39) (xy 190.5 72.39))
     (stroke (width 0) (type default) (color 0 0 0 0))
@@
     (stroke (width 0) (type default) (color 0 0 0 0))
   )
+  (wire (pts (xy 229.87 91.44) (xy 223.52 91.44))
+    (stroke (width 0) (type default) (color 0 0 0 0))
+  )
   (polyline (pts (xy 283.21 71.12) (xy 283.21 13.97))
     (stroke (width 0) (type default) (color 0 0 0 0))
@@
     (stroke (width 0) (type default) (color 0 0 0 0))
   )
+  (wire (pts (xy 254 88.9) (xy 254 91.44))
+    (stroke (width 0) (type default) (color 0 0 0 0))
+  )
   (wire (pts (xy 157.48 40.64) (xy 170.18 40.64))
     (stroke (width 0) (type default) (color 0 0 0 0))
@@
   (polyline (pts (xy 193.04 13.97) (xy 283.21 13.97))
     (stroke (width 0) (type default) (color 0 0 0 0))
+  )
+  (text "3V3 Regulator for the Audio Codec @250mA" (at 217.17 78.74 0)
+    (effects (font (size 1.27 1.27)) (justify left bottom))
+  )
+  (text "3V3 Regulator for the MCU @300mA" (at 214.63 20.32 0)
+    (effects (font (size 1.27 1.27)) (justify left bottom))
   )
   (label "DC_OUT" (at 170.18 40.64 180)
     (effects (font (size 1.27 1.27)) (justify right bottom))
   )
+  (label "DC_OUT" (at 215.9 91.44 0)
+    (effects (font (size 1.27 1.27)) (justify left bottom))
+  )
   (label "DC_OUT" (at 215.9 33.02 0)
     (effects (font (size 1.27 1.27)) (justify left bottom))
@@
     )
     (property "Datasheet" "" (id 3) (at 158.75 90.17 0)
+      (effects (font (size 1.27 1.27)) hide)
+    )
+    (pin "1")
+  )
+  (symbol (lib_id "Device:C_Small") (at 254 95.25 0) (unit 1)
+    (in_bom yes) (on_board yes) (fields_autoplaced)
+    (property "Reference" "C?" (id 0) (at 256.54 93.9862 0)
+      (effects (font (size 1.27 1.27)) (justify left))
+    )
+    (property "Value" "10u" (id 1) (at 256.54 96.5262 0)
+      (effects (font (size 1.27 1.27)) (justify left))
+    )
+    (property "Footprint" "Capacitor_SMD:C_0805_2012Metric" (id 2) (at 254 95.25 0)
+      (effects (font (size 1.27 1.27)) hide)
+    )
+    (property "Datasheet" "~" (id 3) (at 254 95.25 0)
+      (effects (font (size 1.27 1.27)) hide)
+    )
+    (pin "1")
+    (pin "2")
+  )
+  (symbol (lib_id "power:+2V5") (at 254 88.9 0) (unit 1)
+    (in_bom yes) (on_board yes) (fields_autoplaced)
+    (property "Reference" "#PWR?" (id 0) (at 254 92.71 0)
+      (effects (font (size 1.27 1.27)) hide)
+    )
+    (property "Value" "+2V5" (id 1) (at 254 83.82 0))
+    (property "Footprint" "" (id 2) (at 254 88.9 0)
+      (effects (font (size 1.27 1.27)) hide)
+    )
+    (property "Datasheet" "" (id 3) (at 254 88.9 0)
       (effects (font (size 1.27 1.27)) hide)
     )
@@
     (pin "1")
   )
+  (symbol (lib_id "power:GND") (at 254 104.14 0) (unit 1)
+    (in_bom yes) (on_board yes) (fields_autoplaced)
+    (property "Reference" "#PWR?" (id 0) (at 254 110.49 0)
+      (effects (font (size 1.27 1.27)) hide)
+    )
+    (property "Value" "GND" (id 1) (at 254 109.22 0))
+    (property "Footprint" "" (id 2) (at 254 104.14 0)
+      (effects (font (size 1.27 1.27)) hide)
+    )
+    (property "Datasheet" "" (id 3) (at 254 104.14 0)
+      (effects (font (size 1.27 1.27)) hide)
+    )
+    (pin "1")
+  )
   (symbol (lib_id "Device:C_Small") (at 105.41 96.52 0) (unit 1)
     (in_bom yes) (on_board yes) (fields_autoplaced)
@@
     )
     (property "Datasheet" "" (id 3) (at 113.03 105.41 0)
+      (effects (font (size 1.27 1.27)) hide)
+    )
+    (pin "1")
+  )
+  (symbol (lib_id "Device:C_Small") (at 223.52 95.25 0) (unit 1)
+    (in_bom yes) (on_board yes) (fields_autoplaced)
+    (property "Reference" "C?" (id 0) (at 226.06 93.9862 0)
+      (effects (font (size 1.27 1.27)) (justify left))
+    )
+    (property "Value" "10u" (id 1) (at 226.06 96.5262 0)
+      (effects (font (size 1.27 1.27)) (justify left))
+    )
+    (property "Footprint" "Capacitor_SMD:C_0805_2012Metric" (id 2) (at 223.52 95.25 0)
+      (effects (font (size 1.27 1.27)) hide)
+    )
+    (property "Datasheet" "~" (id 3) (at 223.52 95.25 0)
+      (effects (font (size 1.27 1.27)) hide)
+    )
+    (pin "1")
+    (pin "2")
+  )
+  (symbol (lib_id "Regulator_Linear:NCP163ASN280T1G") (at 241.3 93.98 0) (unit 1)
+    (in_bom yes) (on_board yes) (fields_autoplaced)
+    (property "Reference" "U?" (id 0) (at 241.3 83.82 0))
+    (property "Value" "NCP163ASN280T1G" (id 1) (at 241.3 86.36 0))
+    (property "Footprint" "Package_TO_SOT_SMD:SOT-23-5" (id 2) (at 241.3 86.36 0)
+      (effects (font (size 1.27 1.27)) hide)
+    )
+    (property "Datasheet" "https://www.onsemi.com/pdf/datasheet/ncp163-d.pdf" (id 3) (at 241.3 86.36 0)
+      (effects (font (size 1.27 1.27)) hide)
+    )
+    (pin "1")
+    (pin "2")
+    (pin "3")
+    (pin "4")
+    (pin "5")
+  )
+  (symbol (lib_id "power:GND") (at 241.3 104.14 0) (unit 1)
+    (in_bom yes) (on_board yes) (fields_autoplaced)
+    (property "Reference" "#PWR?" (id 0) (at 241.3 110.49 0)
+      (effects (font (size 1.27 1.27)) hide)
+    )
+    (property "Value" "GND" (id 1) (at 241.3 109.22 0))
+    (property "Footprint" "" (id 2) (at 241.3 104.14 0)
+      (effects (font (size 1.27 1.27)) hide)
+    )
+    (property "Datasheet" "" (id 3) (at 241.3 104.14 0)
       (effects (font (size 1.27 1.27)) hide)
     )
@@
       (effects (font (size 1.27 1.27)) hide)
     )
+    (pin "1")
+  )
+  (symbol (lib_id "power:GND") (at 223.52 104.14 0) (unit 1)
+    (in_bom yes) (on_board yes) (fields_autoplaced)
+    (property "Reference" "#PWR?" (id 0) (at 223.52 110.49 0)
+      (effects (font (size 1.27 1.27)) hide)
+    )
+    (property "Value" "GND" (id 1) (at 223.52 109.22 0))
+    (property "Footprint" "" (id 2) (at 223.52 104.14 0)
+      (effects (font (size 1.27 1.27)) hide)
+    )
+    (property "Datasheet" "" (id 3) (at 223.52 104.14 0)
+      (effects (font (size 1.27 1.27)) hide)
+    )

Commit message: update the design
Parts:
- U6: renamed from U?; value NCP163ASN280T1G -> NCP163ASN250T1G
- gave numbers to parts that had none: 2
- renumbered C41 to C28, C42 to C29, C17 to C30, C18 to C32, J3 to J5, J4 to J6, R19 to R15, U2 to U5
