File: hardware/Power-Supply.kicad_sch (KiCad schematic)
At the start: 12 parts, among them J5 CON_USB_GCT_USB4105_REVA, J6 BATT, U4 MCP73831-2-OT, U5 TLV73333PDBV, U6 NCP163ASN250T1G

Commit message: update the design
Parts:
- renumbered C28 to C29, C29 to C30, C30 to C31, C31 to C32, C32 to C33, C33 to C34, J5 to J6, J6 to J7, U4 to U5, U5 to U6, U6 to U7
Changed lines of the file:
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@@
   (symbol (lib_id "power:+BATT") (at 158.75 90.17 0) (mirror y) (unit 1)
     (in_bom yes) (on_board yes) (fields_autoplaced)
-    (property "Reference" "#PWR043" (id 0) (at 158.75 93.98 0)
+    (property "Reference" "#PWR046" (id 0) (at 158.75 93.98 0)
       (effects (font (size 1.27 1.27)) hide)
     )
@@
   (symbol (lib_id "Device:C_Small") (at 254 95.25 0) (unit 1)
     (in_bom yes) (on_board yes) (fields_autoplaced)
-    (property "Reference" "C33" (id 0) (at 256.54 93.9862 0)
+    (property "Reference" "C34" (id 0) (at 256.54 93.9862 0)
       (effects (font (size 1.27 1.27)) (justify left))
     )
@@
   (symbol (lib_id "power:+2V5") (at 254 88.9 0) (unit 1)
     (in_bom yes) (on_board yes) (fields_autoplaced)
-    (property "Reference" "#PWR051" (id 0) (at 254 92.71 0)
+    (property "Reference" "#PWR054" (id 0) (at 254 92.71 0)
       (effects (font (size 1.27 1.27)) hide)
     )
@@
   (symbol (lib_id "Regulator_Linear:TLV73333PDBV") (at 241.3 35.56 0) (unit 1)
     (in_bom yes) (on_board yes) (fields_autoplaced)
-    (property "Reference" "U5" (id 0) (at 241.3 25.4 0))
+    (property "Reference" "U6" (id 0) (at 241.3 25.4 0))
     (property "Value" "TLV73333PDBV" (id 1) (at 241.3 27.94 0))
     (property "Footprint" "Package_TO_SOT_SMD:SOT-23-5" (id 2) (at 241.3 27.305 0)
@@
   (symbol (lib_id "power:GND") (at 124.46 105.41 0) (unit 1)
     (in_bom yes) (on_board yes) (fields_autoplaced)
-    (property "Reference" "#PWR041" (id 0) (at 124.46 111.76 0)
+    (property "Reference" "#PWR044" (id 0) (at 124.46 111.76 0)
       (effects (font (size 1.27 1.27)) hide)
     )
@@
   (symbol (lib_id "power:GND") (at 148.59 104.14 0) (unit 1)
     (in_bom yes) (on_board yes) (fields_autoplaced)
-    (property "Reference" "#PWR042" (id 0) (at 148.59 110.49 0)
+    (property "Reference" "#PWR045" (id 0) (at 148.59 110.49 0)
       (effects (font (size 1.27 1.27)) hide)
     )
@@
   (symbol (lib_id "Device:C_Small") (at 223.52 36.83 0) (unit 1)
     (in_bom yes) (on_board yes) (fields_autoplaced)
-    (property "Reference" "C30" (id 0) (at 226.06 35.5662 0)
+    (property "Reference" "C31" (id 0) (at 226.06 35.5662 0)
       (effects (font (size 1.27 1.27)) (justify left))
     )
@@
   (symbol (lib_id "power:GND") (at 48.26 62.23 0) (unit 1)
     (in_bom yes) (on_board yes) (fields_autoplaced)
-    (property "Reference" "#PWR034" (id 0) (at 48.26 68.58 0)
+    (property "Reference" "#PWR037" (id 0) (at 48.26 68.58 0)
       (effects (font (size 1.27 1.27)) hide)
     )
@@
   (symbol (lib_id "power:+3.3V") (at 254 30.48 0) (unit 1)
     (in_bom yes) (on_board yes) (fields_autoplaced)
-    (property "Reference" "#PWR049" (id 0) (at 254 34.29 0)
+    (property "Reference" "#PWR052" (id 0) (at 254 34.29 0)
       (effects (font (size 1.27 1.27)) hide)
     )
@@
   (symbol (lib_id "power:+BATT") (at 106.68 41.91 0) (unit 1)
     (in_bom yes) (on_board yes) (fields_autoplaced)
-    (property "Reference" "#PWR038" (id 0) (at 106.68 45.72 0)
+    (property "Reference" "#PWR041" (id 0) (at 106.68 45.72 0)
       (effects (font (size 1.27 1.27)) hide)
     )
@@
   (symbol (lib_id "power:GND") (at 254 104.14 0) (unit 1)
     (in_bom yes) (on_board yes) (fields_autoplaced)
-    (property "Reference" "#PWR052" (id 0) (at 254 110.49 0)
+    (property "Reference" "#PWR055" (id 0) (at 254 110.49 0)
       (effects (font (size 1.27 1.27)) hide)
     )
@@
   (symbol (lib_id "Device:C_Small") (at 105.41 96.52 0) (unit 1)
     (in_bom yes) (on_board yes) (fields_autoplaced)
-    (property "Reference" "C28" (id 0) (at 107.95 95.2562 0)
+    (property "Reference" "C29" (id 0) (at 107.95 95.2562 0)
       (effects (font (size 1.27 1.27)) (justify left))
     )
@@
   (symbol (lib_id "power:GND") (at 223.52 45.72 0) (unit 1)
     (in_bom yes) (on_board yes) (fields_autoplaced)
-    (property "Reference" "#PWR045" (id 0) (at 223.52 52.07 0)
+    (property "Reference" "#PWR048" (id 0) (at 223.52 52.07 0)
       (effects (font (size 1.27 1.27)) hide)
     )
@@
   (symbol (lib_id "power:GND") (at 254 45.72 0) (unit 1)
     (in_bom yes) (on_board yes) (fields_autoplaced)
-    (property "Reference" "#PWR050" (id 0) (at 254 52.07 0)
+    (property "Reference" "#PWR053" (id 0) (at 254 52.07 0)
       (effects (font (size 1.27 1.27)) hide)
     )
@@
   (symbol (lib_id "power:VBUS") (at 53.34 22.86 0) (unit 1)
     (in_bom yes) (on_board yes)
-    (property "Reference" "#PWR035" (id 0) (at 53.34 26.67 0)
+    (property "Reference" "#PWR038" (id 0) (at 53.34 26.67 0)
       (effects (font (size 1.27 1.27)) hide)
     )
@@
   (symbol (lib_id "power:GND") (at 113.03 105.41 0) (unit 1)
     (in_bom yes) (on_board yes) (fields_autoplaced)
-    (property "Reference" "#PWR039" (id 0) (at 113.03 111.76 0)
+    (property "Reference" "#PWR042" (id 0) (at 113.03 111.76 0)
       (effects (font (size 1.27 1.27)) hide)
     )
@@
   (symbol (lib_id "Device:C_Small") (at 223.52 95.25 0) (unit 1)
     (in_bom yes) (on_board yes) (fields_autoplaced)
-    (property "Reference" "C31" (id 0) (at 226.06 93.9862 0)
+    (property "Reference" "C32" (id 0) (at 226.06 93.9862 0)
       (effects (font (size 1.27 1.27)) (justify left))
     )
@@
   (symbol (lib_id "Regulator_Linear:NCP163ASN280T1G") (at 241.3 93.98 0) (unit 1)
     (in_bom yes) (on_board yes) (fields_autoplaced)
-    (property "Reference" "U6" (id 0) (at 241.3 83.82 0))
+    (property "Reference" "U7" (id 0) (at 241.3 83.82 0))
     (property "Value" "NCP163ASN250T1G" (id 1) (at 241.3 86.36 0))
     (property "Footprint" "Package_TO_SOT_SMD:SOT-23-5" (id 2) (at 241.3 86.36 0)
@@
   (symbol (lib_id "power:GND") (at 241.3 104.14 0) (unit 1)
     (in_bom yes) (on_board yes) (fields_autoplaced)
-    (property "Reference" "#PWR048" (id 0) (at 241.3 110.49 0)
+    (property "Reference" "#PWR051" (id 0) (at 241.3 110.49 0)
       (effects (font (size 1.27 1.27)) hide)
     )
@@
   (symbol (lib_id "Device:C_Small") (at 254 36.83 0) (unit 1)
     (in_bom yes) (on_board yes) (fields_autoplaced)
-    (property "Reference" "C32" (id 0) (at 256.54 35.5662 0)
+    (property "Reference" "C33" (id 0) (at 256.54 35.5662 0)
       (effects (font (size 1.27 1.27)) (justify left))
     )
@@
   (symbol (lib_id "Connector_Generic:Conn_01x02") (at 168.91 97.79 0) (mirror x) (unit 1)
     (in_bom yes) (on_board yes) (fields_autoplaced)
-    (property "Reference" "J6" (id 0) (at 168.91 88.9 0))
+    (property "Reference" "J7" (id 0) (at 168.91 88.9 0))
     (property "Value" "BATT" (id 1) (at 168.91 91.44 0))
     (property "Footprint" "Connector_JST:JST_EH_S2B-EH_1x02_P2.50mm_Horizontal" (id 2) (at 168.91 97.79 0)
@@
   (symbol (lib_id "1KiCadLib:CON_USB_GCT_USB4105_REVA") (at 24.13 36.83 0) (unit 1)
     (in_bom yes) (on_board yes) (fields_autoplaced)
-    (property "Reference" "J5" (id 0) (at 31.115 19.05 0))
+    (property "Reference" "J6" (id 0) (at 31.115 19.05 0))
     (property "Value" "CON_USB_GCT_USB4105_REVA" (id 1) (at 31.115 21.59 0))
     (property "Footprint" "1KiCadLib:CON_USB_GCT_USB4105_REVA" (id 2) (at 5.08 21.59 0)
@@
   (symbol (lib_id "power:GND") (at 241.3 45.72 0) (unit 1)
     (in_bom yes) (on_board yes) (fields_autoplaced)
-    (property "Reference" "#PWR047" (id 0) (at 241.3 52.07 0)
+    (property "Reference" "#PWR050" (id 0) (at 241.3 52.07 0)
       (effects (font (size 1.27 1.27)) hide)
     )
@@
   (symbol (lib_id "power:VBUS") (at 106.68 26.67 0) (unit 1)
     (in_bom yes) (on_board yes)
-    (property "Reference" "#PWR037" (id 0) (at 106.68 30.48 0)
+    (property "Reference" "#PWR040" (id 0) (at 106.68 30.48 0)
       (effects (font (size 1.27 1.27)) hide)
     )
@@
   (symbol (lib_id "power:GND") (at 105.41 105.41 0) (unit 1)
     (in_bom yes) (on_board yes) (fields_autoplaced)
-    (property "Reference" "#PWR036" (id 0) (at 105.41 111.76 0)
+    (property "Reference" "#PWR039" (id 0) (at 105.41 111.76 0)
       (effects (font (size 1.27 1.27)) hide)
     )
@@
   (symbol (lib_id "power:VBUS") (at 124.46 83.82 0) (unit 1)
     (in_bom yes) (on_board yes)
-    (property "Reference" "#PWR040" (id 0) (at 124.46 87.63 0)
+    (property "Reference" "#PWR043" (id 0) (at 124.46 87.63 0)
       (effects (font (size 1.27 1.27)) hide)
     )
@@
   (symbol (lib_id "power:GND") (at 158.75 104.14 0) (mirror y) (unit 1)
     (in_bom yes) (on_board yes) (fields_autoplaced)
-    (property "Reference" "#PWR044" (id 0) (at 158.75 110.49 0)
+    (property "Reference" "#PWR047" (id 0) (at 158.75 110.49 0)
       (effects (font (size 1.27 1.27)) hide)
     )
@@
   (symbol (lib_id "power:GND") (at 223.52 104.14 0) (unit 1)
     (in_bom yes) (on_board yes) (fields_autoplaced)
-    (property "Reference" "#PWR046" (id 0) (at 223.52 110.49 0)
+    (property "Reference" "#PWR049" (id 0) (at 223.52 110.49 0)
       (effects (font (size 1.27 1.27)) hide)
     )
@@
   (symbol (lib_id "Device:C_Small") (at 148.59 96.52 0) (unit 1)
     (in_bom yes) (on_board yes) (fields_autoplaced)
-    (property "Reference" "C29" (id 0) (at 151.13 95.2562 0)
+    (property "Reference" "C30" (id 0) (at 151.13 95.2562 0)
       (effects (font (size 1.27 1.27)) (justify left))
     )
@@
   (symbol (lib_id "Battery_Management:MCP73831-2-OT") (at 124.46 93.98 0) (unit 1)
     (in_bom yes) (on_board yes) (fields_autoplaced)
-    (property "Reference" "U4" (id 0) (at 126.4794 83.82 0)
-      (effects (font (size 1.27 1.27)) (justify left))
-    )
+    (property "Reference" "U5" (id 0) (at 126.4794 83.82 0)
+      (effects (font (size 1.27 1.27)) (justify left))
+    )
