File: hardware/Power-Supply.kicad_sch (KiCad schematic)
At the start: 12 parts, among them J6 CON_USB_GCT_USB4105_REVA, J7 BATT, U5 MCP73831-2-OT, U6 TLV73333PDBV, U7 NCP163ASN250T1G

Commit message: update the design
Parts:
- added C35, C37, C38: 22u, Capacitor_SMD:C_0805_2012Metric, symbol Device:C_Small
- added C36: 120p, Capacitor_SMD:C_0805_2012Metric, symbol Device:C_Small
- added C39: 100u, Capacitor_SMD:C_0805_2012Metric, symbol Device:C_Small
- added D2: D_Schottky, symbol Device:D_Schottky
- added D3: LED, LED_SMD:LED_0805_2012Metric, symbol Device:LED
- added L1: 2.2uH, symbol Device:L_Small
- added R17: 20k, Resistor_SMD:R_0805_2012Metric, symbol Device:R_Small
- added R18: 5R, symbol Device:R_Small
- added R19, R20, R22: 10K, Resistor_SMD:R_0805_2012Metric, symbol Device:R_Small
- added R21: 1K, Resistor_SMD:R_0805_2012Metric, symbol Device:R_Small
- added U10: TPS2116, Package_TO_SOT_SMD:SOT-23-8, symbol LibraryAudioBoard:TPS2116
- added U8: AP22652W6-7, Package_TO_SOT_SMD:SOT-23-6, symbol LibraryAudioBoard:AP22652W6-7
- added U9: TPS613222ADBV, Package_TO_SOT_SMD:SOT-23-5, symbol Regulator_Switching:TPS613222ADBV
Connections:
- net +BATT: now also U10.6 (VIN2)
- net GND: now also C35.2, C37.2, C38.2, C39.2, D3.1 (K), R17.2, R20.2, U10.1 (GND), U8.2 (GND), U9.2 (GND)
- net VBUS: now also R19.1, U10.3 (VIN1), U10.5 (MODE)
- net DC_OUT renamed MAIN_PWR
- net MAIN_PWR: now also C39.1, R22.1, U10.2 (VOUT), U10.7 (VOUT), U8.1 (IN)
- new net: C36.1, R18.2
- new net: D3.2 (A), R21.2
- new net: R17.1, U8.5 (ILIM)
- new net: D2.2 (A), L1.2, R18.1, U9.1 (SW)
- new net: R22.2, U10.8 (ST)
- new net: R19.2, R20.1, U10.4 (PR1)
- new net BOOST_IN: C35.1, L1.1, U8.6 (OUT)
- new net USB_OTG_EN: U8.3 (EN)
- new net USB_OTG_VBUS: C36.2, C37.1, C38.1, D2.1 (K), R21.1, U9.4 (VOUT)
- no-connect marks 2 -> 4
Other:
- removed sheet PowerSelector
- note added: "Power selector with Power MUX IC"
- note added: "The USB Voltage has the highest priority"
- note added: "USB OTG Power circuit with a Boost IC and Power Switch IC"
- moved on the sheet: C29, C30, J7, R15, U5

Commit message: Update placements
Parts:
- D2: footprint (none) -> Diode_SMD:D_SOD-123
- J7: footprint Connector_JST:JST_EH_S2B-EH_1x02_P2.50mm_Horizontal -> Connector_JST:JST_EH_B2B-EH-A_1x02_P2.50mm_Vertical
- L1: footprint (none) -> Inductor_SMD:L_2010_5025Metric
- R18: footprint (none) -> Diode_SMD:D_0805_2012Metric
Changed lines of the file:
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@@
     (property "Reference" "D2" (id 0) (at 105.7275 146.05 0))
     (property "Value" "D_Schottky" (id 1) (at 105.7275 148.59 0))
-    (property "Footprint" "" (id 2) (at 105.41 152.4 0)
+    (property "Footprint" "Diode_SMD:D_SOD-123" (id 2) (at 105.41 152.4 0)
       (effects (font (size 1.27 1.27)) hide)
     )
@@
     (property "Reference" "R18" (id 0) (at 99.06 142.24 90))
     (property "Value" "5R" (id 1) (at 93.98 142.24 90))
-    (property "Footprint" "" (id 2) (at 96.52 144.78 0)
+    (property "Footprint" "Diode_SMD:D_0805_2012Metric" (id 2) (at 96.52 144.78 0)
       (effects (font (size 1.27 1.27)) hide)
     )
@@
     (property "Reference" "L1" (id 0) (at 88.9 157.48 90))
     (property "Value" "2.2uH" (id 1) (at 88.9 160.02 90))
-    (property "Footprint" "" (id 2) (at 88.9 162.56 0)
+    (property "Footprint" "Inductor_SMD:L_2010_5025Metric" (id 2) (at 88.9 162.56 0)
       (effects (font (size 1.27 1.27)) hide)
     )
@@
     (property "Reference" "J7" (id 0) (at 162.56 92.71 0))
     (property "Value" "BATT" (id 1) (at 162.56 95.25 0))
-    (property "Footprint" "Connector_JST:JST_EH_S2B-EH_1x02_P2.50mm_Horizontal" (id 2) (at 162.56 101.6 0)
-      (effects (font (size 1.27 1.27)) hide)
-    )
+    (property "Footprint" "Connector_JST:JST_EH_B2B-EH-A_1x02_P2.50mm_Vertical" (id 2) (at 162.56 101.6 0)
+      (effects (font (size 1.27 1.27)) hide)
+    )
