File: hardware/PowerSelector.kicad_sch (KiCad schematic)
At the start: 11 parts, among them Q1 DMP2040USD-13, Q2 DMP2040USD-13, Q3 SI2324DS-T1-GE3, Q4 SI2324DS-T1-GE3

Commit message: update the design
Parts:
- renumbered C19 to C34, R5 to R16, R6 to R17, R7 to R18, R8 to R19, R9 to R20, R10 to R21
Changed lines of the file:
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@@
   (symbol (lib_id "power:GND") (at 135.89 129.54 0) (unit 1)
     (in_bom yes) (on_board yes)
-    (property "Reference" "#PWR029" (id 0) (at 135.89 135.89 0)
+    (property "Reference" "#PWR055" (id 0) (at 135.89 135.89 0)
       (effects (font (size 1.27 1.27)) hide)
     )
@@
   (symbol (lib_id "Device:R_Small") (at 114.3 66.04 0) (unit 1)
     (in_bom yes) (on_board yes) (fields_autoplaced)
-    (property "Reference" "R8" (id 0) (at 116.84 64.7699 0)
+    (property "Reference" "R19" (id 0) (at 116.84 64.7699 0)
       (effects (font (size 1.27 1.27)) (justify left))
     )
@@
   (symbol (lib_id "power:GND") (at 113.03 130.81 0) (unit 1)
     (in_bom yes) (on_board yes)
-    (property "Reference" "#PWR027" (id 0) (at 113.03 137.16 0)
+    (property "Reference" "#PWR053" (id 0) (at 113.03 137.16 0)
       (effects (font (size 1.27 1.27)) hide)
     )
@@
   (symbol (lib_id "Device:R_Small") (at 114.3 46.99 0) (unit 1)
     (in_bom yes) (on_board yes) (fields_autoplaced)
-    (property "Reference" "R7" (id 0) (at 116.84 45.7199 0)
+    (property "Reference" "R18" (id 0) (at 116.84 45.7199 0)
       (effects (font (size 1.27 1.27)) (justify left))
     )
@@
   (symbol (lib_id "Device:R_Small") (at 135.89 43.18 0) (unit 1)
     (in_bom yes) (on_board yes) (fields_autoplaced)
-    (property "Reference" "R9" (id 0) (at 138.43 41.9099 0)
+    (property "Reference" "R20" (id 0) (at 138.43 41.9099 0)
       (effects (font (size 1.27 1.27)) (justify left))
     )
@@
   (symbol (lib_id "power:GND") (at 135.89 69.85 0) (unit 1)
     (in_bom yes) (on_board yes)
-    (property "Reference" "#PWR028" (id 0) (at 135.89 76.2 0)
+    (property "Reference" "#PWR054" (id 0) (at 135.89 76.2 0)
       (effects (font (size 1.27 1.27)) hide)
     )
@@
   (symbol (lib_id "Device:C_Small") (at 121.92 124.46 0) (unit 1)
     (in_bom yes) (on_board yes) (fields_autoplaced)
-    (property "Reference" "C19" (id 0) (at 124.46 123.1962 0)
+    (property "Reference" "C34" (id 0) (at 124.46 123.1962 0)
       (effects (font (size 1.27 1.27)) (justify left))
     )
@@
   (symbol (lib_id "Device:R_Small") (at 135.89 92.71 0) (unit 1)
     (in_bom yes) (on_board yes) (fields_autoplaced)
-    (property "Reference" "R10" (id 0) (at 138.43 91.4399 0)
+    (property "Reference" "R21" (id 0) (at 138.43 91.4399 0)
       (effects (font (size 1.27 1.27)) (justify left))
     )
@@
   (symbol (lib_id "Device:R_Small") (at 113.03 93.98 0) (unit 1)
     (in_bom yes) (on_board yes) (fields_autoplaced)
-    (property "Reference" "R5" (id 0) (at 115.57 92.7099 0)
+    (property "Reference" "R16" (id 0) (at 115.57 92.7099 0)
       (effects (font (size 1.27 1.27)) (justify left))
     )
@@
   (symbol (lib_id "Device:R_Small") (at 113.03 124.46 0) (unit 1)
     (in_bom yes) (on_board yes)
-    (property "Reference" "R6" (id 0) (at 114.3 123.19 0)
-      (effects (font (size 1.27 1.27)) (justify left))
-    )
+    (property "Reference" "R17" (id 0) (at 114.3 123.19 0)
+      (effects (font (size 1.27 1.27)) (justify left))
+    )

Commit message: update the design
Parts:
- renumbered C34 to C35
Changed lines of the file:
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@@
   (symbol (lib_id "power:GND") (at 135.89 129.54 0) (unit 1)
     (in_bom yes) (on_board yes)
-    (property "Reference" "#PWR055" (id 0) (at 135.89 135.89 0)
+    (property "Reference" "#PWR058" (id 0) (at 135.89 135.89 0)
       (effects (font (size 1.27 1.27)) hide)
     )
@@
   (symbol (lib_id "power:GND") (at 113.03 130.81 0) (unit 1)
     (in_bom yes) (on_board yes)
-    (property "Reference" "#PWR053" (id 0) (at 113.03 137.16 0)
+    (property "Reference" "#PWR056" (id 0) (at 113.03 137.16 0)
       (effects (font (size 1.27 1.27)) hide)
     )
@@
   (symbol (lib_id "power:GND") (at 135.89 69.85 0) (unit 1)
     (in_bom yes) (on_board yes)
-    (property "Reference" "#PWR054" (id 0) (at 135.89 76.2 0)
+    (property "Reference" "#PWR057" (id 0) (at 135.89 76.2 0)
       (effects (font (size 1.27 1.27)) hide)
     )
@@
   (symbol (lib_id "Device:C_Small") (at 121.92 124.46 0) (unit 1)
     (in_bom yes) (on_board yes) (fields_autoplaced)
-    (property "Reference" "C34" (id 0) (at 124.46 123.1962 0)
+    (property "Reference" "C35" (id 0) (at 124.46 123.1962 0)
       (effects (font (size 1.27 1.27)) (justify left))
     )
