File: hardware/audio-codec.kicad_sch (KiCad schematic)
At the start: 0 parts

Commit message: update the file
Parts:
- added C? (x2): 22p, Capacitor_SMD:C_0603_1608Metric, symbol Device:C_Small
- added C? (x5): 100n, Capacitor_SMD:C_0603_1608Metric, symbol Device:C_Small
- added C?: 10u, Capacitor_SMD:C_0805_2012Metric, symbol Device:C_Small
- added C? (x3): 1u, Capacitor_SMD:C_0805_2012Metric, symbol Device:C_Small
- added C? (x2): 150p, Capacitor_SMD:C_0603_1608Metric, symbol Device:C_Small
- added C? (x2): 1u(X7R), symbol Device:C_Small
- added R? (x2): 51R, Resistor_SMD:R_0805_2012Metric, symbol Device:R_Small
- added R?: 10K, Resistor_SMD:R_0805_2012Metric, symbol Device:R_Small
- added U?: CS42L51-CNZ, Package_DFN_QFN:QFN-32-1EP_5x5mm_P0.5mm_EP3.1x3.1mm, symbol LibraryAudioBoard:CS42L51-CNZ
Connections:
- new net: C?.1, U?.10 (AOUTB)
- new net: C?.1, U?.11 (AOUTA)
- new net: C?.1, U?.14 (DAC_FILT+)
- new net: C?.1, U?.15 (VQ)
- new net: C?.1, U?.16 (ADC_FILT+)
- new net: C?.1, U?.21 (AFILTA)
- new net: C?.1, U?.22 (AFILTB)
- new net: C?.1, U?.6 (FLYP)
- new net: C?.2, U?.8 (FLYN)
- new net: C?.1, U?.9 (VSS_HP)
- new net: C?.2, R?.1 (x2)
- new net +2V5: C?.1, C?.1, C?.1, C?.1, C?.1, U?.12 (VA), U?.27 (VD), U?.5 (VA_HP)
- new net +3.3V: C?.1, R?.1, U?.26 (VL)
- new net GND: C?.2, C?.2, C?.2, C?.2, C?.2, C?.2, C?.2, C?.2, C?.2, C?.2, C?.2, C?.2, R?.2, R?.2, U?.13 (AGND), U?.28 (DGND), U?.33 (EXP), U?.7 (GND_HP)
- new net MCLK: U?.30 (MCLK)
- new net SCL: U?.1 (LRCK), U?.3 (SCL/CCLK(I2S/~{LJ}))
- new net SCLK: U?.31 (SCLK)
- new net SDA: U?.2 (SDA/CDIN(MCLKDIV2))
- new net SDIN: U?.32 (SDIN)
- new net SDOUT: U?.29 (SDOUT(M/~{S}))
- new net ~{RST}: R?.2, U?.25 (~{RESET})

Commit message: update the file
Parts:
- added C3: 1u, Capacitor_SMD:C_0805_2012Metric, symbol Device:C_Small
- added J2: AudioJack3_Ground, symbol Connector:AudioJack3_Ground
- added R3: 100R, Resistor_SMD:R_0805_2012Metric, symbol Device:R_Small
- gave numbers to parts that had none: 19
Connections:
- net GND: now also U1.4 (AD0/~{CS}(DEM)), J2.G, J2.T
- net at C1.1, U1.10 (AOUTB): now also J2.R
- net at C2.1, U1.11 (AOUTA): now also J2.S
- net at U1.23 (AIN1A): now also U1.24 (AIN1B), R3.2
- new net: C3.2, R3.1

Commit message: update the design
Connections:
- no-connect marks 0 -> 4
Other:
- moved on the sheet: C3, R3
Changed lines of the file:
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@@
   (junction (at 186.69 52.07) (diameter 0) (color 0 0 0 0)
   )
+  (no_connect (at 134.62 100.33))
+  (no_connect (at 134.62 107.95))
+  (no_connect (at 134.62 105.41))
+  (no_connect (at 134.62 102.87))
   (wire (pts (xy 193.04 53.34) (xy 193.04 52.07))
     (stroke (width 0) (type default) (color 0 0 0 0))
@@
     (stroke (width 0) (type default) (color 0 0 0 0))
   )
-  (wire (pts (xy 125.73 96.52) (xy 130.81 96.52))
+  (wire (pts (xy 127 96.52) (xy 130.81 96.52))
     (stroke (width 0) (type default) (color 0 0 0 0))
   )
@@
     (stroke (width 0) (type default) (color 0 0 0 0))
   )
+  (wire (pts (xy 96.52 96.52) (xy 106.68 96.52))
+    (stroke (width 0) (type default) (color 0 0 0 0))
+  )
   (wire (pts (xy 224.79 80.01) (xy 185.42 80.01))
     (stroke (width 0) (type default) (color 0 0 0 0))
@@
     (stroke (width 0) (type default) (color 0 0 0 0))
   )
-  (wire (pts (xy 115.57 96.52) (xy 120.65 96.52))
+  (wire (pts (xy 111.76 96.52) (xy 121.92 96.52))
     (stroke (width 0) (type default) (color 0 0 0 0))
   )
@@
     (stroke (width 0) (type default) (color 0 0 0 0))
   )
-  (wire (pts (xy 185.42 95.25) (xy 190.5 95.25))
+  (wire (pts (xy 185.42 95.25) (xy 193.04 95.25))
     (stroke (width 0) (type default) (color 0 0 0 0))
   )
@@
     (stroke (width 0) (type default) (color 0 0 0 0))
   )
-  (wire (pts (xy 185.42 92.71) (xy 190.5 92.71))
+  (wire (pts (xy 185.42 92.71) (xy 193.04 92.71))
     (stroke (width 0) (type default) (color 0 0 0 0))
   )
@@
     (stroke (width 0) (type default) (color 0 0 0 0))
   )
-  (wire (pts (xy 185.42 100.33) (xy 189.23 100.33))
+  (wire (pts (xy 185.42 100.33) (xy 190.5 100.33))
     (stroke (width 0) (type default) (color 0 0 0 0))
   )
@@
     (stroke (width 0) (type default) (color 0 0 0 0))
   )
-  (wire (pts (xy 189.23 100.33) (xy 189.23 101.6))
+  (wire (pts (xy 190.5 100.33) (xy 190.5 101.6))
     (stroke (width 0) (type default) (color 0 0 0 0))
   )
@@
     (effects (font (size 1.27 1.27)) (justify right))
   )
-  (hierarchical_label "SCL" (shape input) (at 190.5 92.71 0)
+  (hierarchical_label "SCL" (shape input) (at 193.04 92.71 0)
     (effects (font (size 1.27 1.27)) (justify left))
   )
@@
     (effects (font (size 1.27 1.27)) (justify right))
   )
-  (hierarchical_label "SDA" (shape bidirectional) (at 190.5 95.25 0)
+  (hierarchical_label "SDA" (shape bidirectional) (at 193.04 95.25 0)
     (effects (font (size 1.27 1.27)) (justify left))
   )
@@
     (effects (font (size 1.27 1.27)) (justify right))
   )
-  (symbol (lib_id "Device:R_Small") (at 123.19 96.52 90) (unit 1)
-    (in_bom yes) (on_board yes)
-    (property "Reference" "R3" (id 0) (at 121.92 93.98 90)
-      (effects (font (size 1.27 1.27)) (justify left))
-    )
-    (property "Value" "100R" (id 1) (at 127 93.98 90)
-      (effects (font (size 1.27 1.27)) (justify left))
-    )
-    (property "Footprint" "Resistor_SMD:R_0805_2012Metric" (id 2) (at 123.19 96.52 0)
-      (effects (font (size 1.27 1.27)) hide)
-    )
-    (property "Datasheet" "~" (id 3) (at 123.19 96.52 0)
+  (symbol (lib_id "Device:R_Small") (at 124.46 96.52 90) (unit 1)
+    (in_bom yes) (on_board yes)
+    (property "Reference" "R3" (id 0) (at 119.38 95.25 90)
+      (effects (font (size 1.27 1.27)) (justify left))
+    )
+    (property "Value" "100R" (id 1) (at 128.27 93.98 90)
+      (effects (font (size 1.27 1.27)) (justify left))
+    )
+    (property "Footprint" "Resistor_SMD:R_0805_2012Metric" (id 2) (at 124.46 96.52 0)
+      (effects (font (size 1.27 1.27)) hide)
+    )
+    (property "Datasheet" "~" (id 3) (at 124.46 96.52 0)
       (effects (font (size 1.27 1.27)) hide)
     )
@@
   )
   (symbol (lib_id "Device:C_Small") (at 224.79 91.44 0) (unit 1)
-    (in_bom yes) (on_board yes) (fields_autoplaced)
-    (property "Reference" "C13" (id 0) (at 227.33 90.1762 0)
-      (effects (font (size 1.27 1.27)) (justify left))
-    )
-    (property "Value" "10u" (id 1) (at 227.33 92.7162 0)
+    (in_bom yes) (on_board yes)
+    (property "Reference" "C13" (id 0) (at 224.79 88.9 0)
+      (effects (font (size 1.27 1.27)) (justify left))
+    )
+    (property "Value" "10u" (id 1) (at 224.79 93.98 0)
       (effects (font (size 1.27 1.27)) (justify left))
     )
@@
   )
   (symbol (lib_id "Device:C_Small") (at 214.63 66.04 0) (unit 1)
-    (in_bom yes) (on_board yes) (fields_autoplaced)
+    (in_bom yes) (on_board yes)
     (property "Reference" "C10" (id 0) (at 217.17 64.7762 0)
       (effects (font (size 1.27 1.27)) (justify left))
@@
   )
   (symbol (lib_id "Device:C_Small") (at 190.5 111.76 0) (unit 1)
-    (in_bom yes) (on_board yes) (fields_autoplaced)
-    (property "Reference" "C7" (id 0) (at 193.04 110.4962 0)
-      (effects (font (size 1.27 1.27)) (justify left))
-    )
-    (property "Value" "1u(X7R)" (id 1) (at 193.04 113.0362 0)
+    (in_bom yes) (on_board yes)
+    (property "Reference" "C7" (id 0) (at 191.77 110.49 0)
+      (effects (font (size 1.27 1.27)) (justify left))
+    )
+    (property "Value" "1u(X7R)" (id 1) (at 191.77 113.03 0)
       (effects (font (size 1.27 1.27)) (justify left))
     )
@@
     (pin "2")
   )
-  (symbol (lib_id "power:GND") (at 189.23 101.6 0) (unit 1)
-    (in_bom yes) (on_board yes)
-    (property "Reference" "#PWR09" (id 0) (at 189.23 107.95 0)
-      (effects (font (size 1.27 1.27)) hide)
-    )
-    (property "Value" "GND" (id 1) (at 189.23 105.41 0))
-    (property "Footprint" "" (id 2) (at 189.23 101.6 0)
-      (effects (font (size 1.27 1.27)) hide)
-    )
-    (property "Datasheet" "" (id 3) (at 189.23 101.6 0)
+  (symbol (lib_id "power:GND") (at 190.5 101.6 0) (unit 1)
+    (in_bom yes) (on_board yes)
+    (property "Reference" "#PWR09" (id 0) (at 190.5 107.95 0)
+      (effects (font (size 1.27 1.27)) hide)
+    )
+    (property "Value" "GND" (id 1) (at 190.5 105.41 0))
+    (property "Footprint" "" (id 2) (at 190.5 101.6 0)
+      (effects (font (size 1.27 1.27)) hide)
+    )
+    (property "Datasheet" "" (id 3) (at 190.5 101.6 0)
       (effects (font (size 1.27 1.27)) hide)
     )
@@
   )
   (symbol (lib_id "Device:C_Small") (at 215.9 91.44 0) (unit 1)
-    (in_bom yes) (on_board yes) (fields_autoplaced)
-    (property "Reference" "C11" (id 0) (at 218.44 90.1762 0)
-      (effects (font (size 1.27 1.27)) (justify left))
-    )
-    (property "Value" "1u" (id 1) (at 218.44 92.7162 0)
+    (in_bom yes) (on_board yes)
+    (property "Reference" "C11" (id 0) (at 215.9 88.9 0)
+      (effects (font (size 1.27 1.27)) (justify left))
+    )
+    (property "Value" "1u" (id 1) (at 215.9 93.98 0)
       (effects (font (size 1.27 1.27)) (justify left))
     )
@@
   )
   (symbol (lib_id "Device:C_Small") (at 208.28 91.44 0) (unit 1)
-    (in_bom yes) (on_board yes) (fields_autoplaced)
-    (property "Reference" "C9" (id 0) (at 210.82 90.1762 0)
-      (effects (font (size 1.27 1.27)) (justify left))
-    )
-    (property "Value" "1u" (id 1) (at 210.82 92.7162 0)
+    (in_bom yes) (on_board yes)
+    (property "Reference" "C9" (id 0) (at 208.28 88.9 0)
+      (effects (font (size 1.27 1.27)) (justify left))
+    )
+    (property "Value" "1u" (id 1) (at 208.28 93.98 0)
       (effects (font (size 1.27 1.27)) (justify left))
     )
@@
     (pin "2")
   )
-  (symbol (lib_id "Device:C_Small") (at 113.03 96.52 90) (unit 1)
-    (in_bom yes) (on_board yes)
-    (property "Reference" "C3" (id 0) (at 115.57 95.25 90))
-    (property "Value" "1u" (id 1) (at 110.49 95.25 90))
-    (property "Footprint" "Capacitor_SMD:C_0805_2012Metric" (id 2) (at 113.03 96.52 0)
-      (effects (font (size 1.27 1.27)) hide)
-    )
-    (property "Datasheet" "~" (id 3) (at 113.03 96.52 0)
-      (effects (font (size 1.27 1.27)) hide)
-    )
+  (symbol (lib_id "Device:C_Small") (at 109.22 96.52 90) (unit 1)
+    (in_bom yes) (on_board yes)
+    (property "Reference" "C3" (id 0) (at 111.76 95.25 90))
+    (property "Value" "1u" (id 1) (at 106.68 95.25 90))
+    (property "Footprint" "Capacitor_SMD:C_0805_2012Metric" (id 2) (at 109.22 96.52 0)
+      (effects (font (size 1.27 1.27)) hide)
+    )
+    (property "Datasheet" "~" (id 3) (at 109.22 96.52 0)
+      (effects (font (size 1.27 1.27)) hide)
+    )

Commit message: update the design
Parts:
- C6, C7: footprint (none) -> Capacitor_SMD:C_0603_1608Metric
Changed lines of the file:
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@@
       (effects (font (size 1.27 1.27)) (justify left))
     )
-    (property "Footprint" "" (id 2) (at 190.5 111.76 0)
+    (property "Footprint" "Capacitor_SMD:C_0603_1608Metric" (id 2) (at 190.5 111.76 0)
       (effects (font (size 1.27 1.27)) hide)
     )
@@
       (effects (font (size 1.27 1.27)) (justify left))
     )
-    (property "Footprint" "" (id 2) (at 129.54 68.58 0)
+    (property "Footprint" "Capacitor_SMD:C_0603_1608Metric" (id 2) (at 129.54 68.58 0)
       (effects (font (size 1.27 1.27)) hide)
     )

Commit message: update the design
Connections:
- net SCL: no longer U1.1 (LRCK)
- new net LRCK: U1.1 (LRCK)
Changed lines of the file:
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@@
     (stroke (width 0) (type default) (color 0 0 0 0))
   )
-  (wire (pts (xy 128.27 74.93) (xy 134.62 74.93))
+  (wire (pts (xy 121.92 74.93) (xy 134.62 74.93))
     (stroke (width 0) (type default) (color 0 0 0 0))
   )
@@
     (effects (font (size 1.27 1.27)) (justify right))
   )
-  (hierarchical_label "SCL" (shape input) (at 128.27 74.93 180)
+  (hierarchical_label "LRCK" (shape input) (at 121.92 74.93 180)
     (effects (font (size 1.27 1.27)) (justify right))
   )

Commit message: update the design
Parts:
- added R?: 10K, Resistor_SMD:R_0805_2012Metric, symbol Device:R_Small
Connections:
- net GND: now also R?.1
- net SDOUT renamed M/~{S}
- net M/~{S}: now also R?.2
Other:
- moved on the sheet: C3, R3
Changed lines of the file:
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@@
   (junction (at 99.06 115.57) (diameter 0) (color 0 0 0 0)
   )
+  (junction (at 130.81 96.52) (diameter 0) (color 0 0 0 0)
+  )
   (junction (at 106.68 113.03) (diameter 0) (color 0 0 0 0)
   )
@@
   (junction (at 190.5 120.65) (diameter 0) (color 0 0 0 0)
   )
-  (junction (at 130.81 96.52) (diameter 0) (color 0 0 0 0)
-  )
   (junction (at 214.63 69.85) (diameter 0) (color 0 0 0 0)
   )
+  (junction (at 134.62 90.17) (diameter 0) (color 0 0 0 0)
+  )
   (junction (at 207.01 62.23) (diameter 0) (color 0 0 0 0)
   )
@@
   )
   (junction (at 190.5 118.11) (diameter 0) (color 0 0 0 0)
+  )
+  (junction (at 129.54 90.17) (diameter 0) (color 0 0 0 0)
   )
   (junction (at 240.03 62.23) (diameter 0) (color 0 0 0 0)
@@
     (stroke (width 0) (type default) (color 0 0 0 0))
   )
+  (wire (pts (xy 127 102.87) (xy 129.54 102.87))
+    (stroke (width 0) (type default) (color 0 0 0 0))
+  )
+  (wire (pts (xy 248.92 68.58) (xy 248.92 69.85))
+    (stroke (width 0) (type default) (color 0 0 0 0))
+  )
+  (wire (pts (xy 185.42 64.77) (xy 207.01 64.77))
+    (stroke (width 0) (type default) (color 0 0 0 0))
+  )
   (wire (pts (xy 130.81 96.52) (xy 130.81 97.79))
     (stroke (width 0) (type default) (color 0 0 0 0))
   )
-  (wire (pts (xy 248.92 68.58) (xy 248.92 69.85))
-    (stroke (width 0) (type default) (color 0 0 0 0))
-  )
-  (wire (pts (xy 185.42 64.77) (xy 207.01 64.77))
-    (stroke (width 0) (type default) (color 0 0 0 0))
-  )
   (wire (pts (xy 186.69 50.8) (xy 186.69 52.07))
     (stroke (width 0) (type default) (color 0 0 0 0))
@@
     (stroke (width 0) (type default) (color 0 0 0 0))
   )
+  (wire (pts (xy 138.43 90.17) (xy 134.62 90.17))
+    (stroke (width 0) (type default) (color 0 0 0 0))
+  )
   (wire (pts (xy 127 129.54) (xy 127 130.81))
     (stroke (width 0) (type default) (color 0 0 0 0))
@@
     (stroke (width 0) (type default) (color 0 0 0 0))
   )
+  (wire (pts (xy 118.11 93.98) (xy 120.65 93.98))
+    (stroke (width 0) (type default) (color 0 0 0 0))
+  )
   (wire (pts (xy 134.62 69.85) (xy 133.35 69.85))
     (stroke (width 0) (type default) (color 0 0 0 0))
   )
-  (wire (pts (xy 127 96.52) (xy 130.81 96.52))
+  (wire (pts (xy 129.54 90.17) (xy 134.62 90.17))
     (stroke (width 0) (type default) (color 0 0 0 0))
   )
@@
     (stroke (width 0) (type default) (color 0 0 0 0))
   )
+  (wire (pts (xy 121.92 90.17) (xy 129.54 90.17))
+    (stroke (width 0) (type default) (color 0 0 0 0))
+  )
   (wire (pts (xy 190.5 123.19) (xy 190.5 120.65))
     (stroke (width 0) (type default) (color 0 0 0 0))
@@
     (stroke (width 0) (type default) (color 0 0 0 0))
   )
+  (wire (pts (xy 129.54 102.87) (xy 129.54 96.52))
+    (stroke (width 0) (type default) (color 0 0 0 0))
+  )
   (wire (pts (xy 190.5 115.57) (xy 190.5 118.11))
     (stroke (width 0) (type default) (color 0 0 0 0))
@@
     (stroke (width 0) (type default) (color 0 0 0 0))
   )
+  (wire (pts (xy 129.54 96.52) (xy 130.81 96.52))
+    (stroke (width 0) (type default) (color 0 0 0 0))
+  )
   (wire (pts (xy 240.03 68.58) (xy 240.03 69.85))
     (stroke (width 0) (type default) (color 0 0 0 0))
@@
     (stroke (width 0) (type default) (color 0 0 0 0))
   )
-  (wire (pts (xy 96.52 96.52) (xy 106.68 96.52))
-    (stroke (width 0) (type default) (color 0 0 0 0))
-  )
   (wire (pts (xy 224.79 80.01) (xy 185.42 80.01))
     (stroke (width 0) (type default) (color 0 0 0 0))
@@
     (stroke (width 0) (type default) (color 0 0 0 0))
   )
-  (wire (pts (xy 111.76 96.52) (xy 121.92 96.52))
-    (stroke (width 0) (type default) (color 0 0 0 0))
-  )
   (wire (pts (xy 127 123.19) (xy 134.62 123.19))
     (stroke (width 0) (type default) (color 0 0 0 0))
@@
     (stroke (width 0) (type default) (color 0 0 0 0))
   )
+  (wire (pts (xy 129.54 93.98) (xy 129.54 90.17))
+    (stroke (width 0) (type default) (color 0 0 0 0))
+  )
   (wire (pts (xy 127 124.46) (xy 127 123.19))
     (stroke (width 0) (type default) (color 0 0 0 0))
@@
     (stroke (width 0) (type default) (color 0 0 0 0))
   )
+  (wire (pts (xy 125.73 93.98) (xy 129.54 93.98))
+    (stroke (width 0) (type default) (color 0 0 0 0))
+  )
   (wire (pts (xy 64.77 123.19) (xy 64.77 124.46))
     (stroke (width 0) (type default) (color 0 0 0 0))
   )
+  (wire (pts (xy 114.3 102.87) (xy 121.92 102.87))
+    (stroke (width 0) (type default) (color 0 0 0 0))
+  )
   (wire (pts (xy 121.92 74.93) (xy 134.62 74.93))
     (stroke (width 0) (type default) (color 0 0 0 0))
@@
   )
   (wire (pts (xy 99.06 118.11) (xy 99.06 115.57))
-    (stroke (width 0) (type default) (color 0 0 0 0))
-  )
-  (wire (pts (xy 121.92 90.17) (xy 134.62 90.17))
     (stroke (width 0) (type default) (color 0 0 0 0))
   )
@@
     (effects (font (size 1.27 1.27)) (justify left))
   )
-  (hierarchical_label "SDOUT" (shape output) (at 121.92 90.17 180)
+  (hierarchical_label "M{slash}~{S}" (shape output) (at 121.92 90.17 180)
     (effects (font (size 1.27 1.27)) (justify right))
   )
@@
     (effects (font (size 1.27 1.27)) (justify right))
   )
-  (symbol (lib_id "Device:R_Small") (at 124.46 96.52 90) (unit 1)
-    (in_bom yes) (on_board yes)
-    (property "Reference" "R3" (id 0) (at 119.38 95.25 90)
-      (effects (font (size 1.27 1.27)) (justify left))
-    )
-    (property "Value" "100R" (id 1) (at 128.27 93.98 90)
-      (effects (font (size 1.27 1.27)) (justify left))
-    )
-    (property "Footprint" "Resistor_SMD:R_0805_2012Metric" (id 2) (at 124.46 96.52 0)
-      (effects (font (size 1.27 1.27)) hide)
-    )
-    (property "Datasheet" "~" (id 3) (at 124.46 96.52 0)
+  (symbol (lib_id "Device:R_Small") (at 124.46 102.87 90) (unit 1)
+    (in_bom yes) (on_board yes)
+    (property "Reference" "R3" (id 0) (at 119.38 101.6 90)
+      (effects (font (size 1.27 1.27)) (justify left))
+    )
+    (property "Value" "100R" (id 1) (at 128.27 100.33 90)
+      (effects (font (size 1.27 1.27)) (justify left))
+    )
+    (property "Footprint" "Resistor_SMD:R_0805_2012Metric" (id 2) (at 124.46 102.87 0)
+      (effects (font (size 1.27 1.27)) hide)
+    )
+    (property "Datasheet" "~" (id 3) (at 124.46 102.87 0)
       (effects (font (size 1.27 1.27)) hide)
     )
@@
     (pin "1")
   )
+  (symbol (lib_id "power:GND") (at 118.11 93.98 0) (unit 1)
+    (in_bom yes) (on_board yes)
+    (property "Reference" "#PWR?" (id 0) (at 118.11 100.33 0)
+      (effects (font (size 1.27 1.27)) hide)
+    )
+    (property "Value" "GND" (id 1) (at 115.57 93.98 0))
+    (property "Footprint" "" (id 2) (at 118.11 93.98 0)
+      (effects (font (size 1.27 1.27)) hide)
+    )
+    (property "Datasheet" "" (id 3) (at 118.11 93.98 0)
+      (effects (font (size 1.27 1.27)) hide)
+    )
+    (pin "1")
+  )
   (symbol (lib_id "Device:C_Small") (at 214.63 66.04 0) (unit 1)
     (in_bom yes) (on_board yes)
@@
     (pin "2")
   )
-  (symbol (lib_id "Device:C_Small") (at 109.22 96.52 90) (unit 1)
-    (in_bom yes) (on_board yes)
-    (property "Reference" "C3" (id 0) (at 111.76 95.25 90))
-    (property "Value" "1u" (id 1) (at 106.68 95.25 90))
-    (property "Footprint" "Capacitor_SMD:C_0805_2012Metric" (id 2) (at 109.22 96.52 0)
-      (effects (font (size 1.27 1.27)) hide)
-    )
-    (property "Datasheet" "~" (id 3) (at 109.22 96.52 0)
+  (symbol (lib_id "Device:C_Small") (at 111.76 102.87 90) (unit 1)
+    (in_bom yes) (on_board yes)
+    (property "Reference" "C3" (id 0) (at 114.3 101.6 90))
+    (property "Value" "1u" (id 1) (at 109.22 101.6 90))
+    (property "Footprint" "Capacitor_SMD:C_0805_2012Metric" (id 2) (at 111.76 102.87 0)
+      (effects (font (size 1.27 1.27)) hide)
+    )
+    (property "Datasheet" "~" (id 3) (at 111.76 102.87 0)
       (effects (font (size 1.27 1.27)) hide)
     )
@@
       (effects (font (size 1.27 1.27)) hide)
     )
+    (pin "1")
+    (pin "2")
+  )
+  (symbol (lib_id "Device:R_Small") (at 123.19 93.98 90) (unit 1)
+    (in_bom yes) (on_board yes)
+    (property "Reference" "R?" (id 0) (at 120.65 92.71 90)
+      (effects (font (size 1.27 1.27)) (justify left))
+    )
+    (property "Value" "10K" (id 1) (at 129.54 92.71 90)
+      (effects (font (size 1.27 1.27)) (justify left))
+    )
+    (property "Footprint" "Resistor_SMD:R_0805_2012Metric" (id 2) (at 123.19 93.98 0)
+      (effects (font (size 1.27 1.27)) hide)
+    )
+    (property "Datasheet" "~" (id 3) (at 123.19 93.98 0)
+      (effects (font (size 1.27 1.27)) hide)
+    )

Commit message: update the design
Parts:
- added J?: MIC, Connector_PinSocket_2.54mm:PinSocket_1x02_P2.54mm_Vertical, symbol Connector_Generic:Conn_01x02
- J4: renamed from J2; footprint (none) -> Connector_Audio:Jack_3.5mm_CUI_SJ-3523-SMT_Horizontal
- gave numbers to parts that had none: 1
- renumbered C1 to C12, C2 to C13, C3 to C14, C4 to C15, C5 to C16, C6 to C17, C7 to C18, C8 to C19, C9 to C20, C10 to C21, C11 to C22, C12 to C23, C13 to C24, C14 to C25, C15 to C26, C16 to C27, R1 to R10, R2 to R11, R3 to R13, R4 to R14, U1 to U3
Connections:
- net GND: now also J?.2 (Pin_2)
- net at C14.1: now also J?.1 (Pin_1)

Commit message: update the design
Parts:
- gave numbers to parts that had none: 1
- renumbered C12 to C13, C13 to C14, C14 to C15, C15 to C16, C16 to C17, C17 to C18, C18 to C19, C19 to C20, C20 to C21, C21 to C22, C22 to C23, C23 to C24, C24 to C25, C25 to C26, C26 to C27, C27 to C28, U3 to U4
