File: hardware/audio-codec.kicad_sch (KiCad schematic)
At the start: 24 parts, among them J4 AudioJack3_Ground, J5 MIC, U4 CS42L51-CNZ

Commit message: update the design
Parts:
- removed J4: AudioJack3_Ground, Connector_Audio:Jack_3.5mm_CUI_SJ-3523-SMT_Horizontal, symbol Connector:AudioJack3_Ground
- added J4: SJ-3523-SMT-TR, LibraryAudioBoard:CUI_SJ-3523-SMT-TR, symbol LibraryAudioBoard:SJ-3523-SMT-TR
Connections:
- net GND: now also J4.2
- net at C13.1, U4.10 (AOUTB): now also J4.3
- net at C14.1, U4.11 (AOUTA): now also J4.1
Changed lines of the file:
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@@
-    (stroke (width 0) (type default) (color 0 0 0 0))
-  )
-  (wire (pts (xy 64.77 123.19) (xy 64.77 124.46))
     (stroke (width 0) (type default) (color 0 0 0 0))
   )
@@
     (pin "2")
   )
-  (symbol (lib_id "power:GND") (at 64.77 124.46 0) (unit 1)
-    (in_bom yes) (on_board yes)
-    (property "Reference" "#PWR019" (id 0) (at 64.77 130.81 0)
-      (effects (font (size 1.27 1.27)) hide)
-    )
-    (property "Value" "GND" (id 1) (at 64.77 128.27 0))
-    (property "Footprint" "" (id 2) (at 64.77 124.46 0)
-      (effects (font (size 1.27 1.27)) hide)
-    )
-    (property "Datasheet" "" (id 3) (at 64.77 124.46 0)
-      (effects (font (size 1.27 1.27)) hide)
-    )
-    (pin "1")
-  )
   (symbol (lib_id "Device:C_Small") (at 99.06 120.65 0) (unit 1)
     (in_bom yes) (on_board yes) (fields_autoplaced)
@@
     (pin "1")
   )
-  (symbol (lib_id "Connector:AudioJack3_Ground") (at 64.77 115.57 0) (unit 1)
-    (in_bom yes) (on_board yes) (fields_autoplaced)
-    (property "Reference" "J4" (id 0) (at 62.865 106.68 0))
-    (property "Value" "AudioJack3_Ground" (id 1) (at 62.865 109.22 0))
-    (property "Footprint" "Connector_Audio:Jack_3.5mm_CUI_SJ-3523-SMT_Horizontal" (id 2) (at 64.77 115.57 0)
-      (effects (font (size 1.27 1.27)) hide)
-    )
-    (property "Datasheet" "~" (id 3) (at 64.77 115.57 0)
-      (effects (font (size 1.27 1.27)) hide)
-    )
-    (pin "G")
-    (pin "R")
-    (pin "S")
-    (pin "T")
-  )
   (symbol (lib_id "Device:R_Small") (at 133.35 58.42 0) (unit 1)
     (in_bom yes) (on_board yes)
@@
       (effects (font (size 1.27 1.27)) hide)
     )
-    (property "Value" "GND" (id 1) (at 115.57 93.98 0))
+    (property "Value" "GND" (id 1) (at 118.11 97.79 0))
     (property "Footprint" "" (id 2) (at 118.11 93.98 0)
       (effects (font (size 1.27 1.27)) hide)
@@
     (pin "1")
   )
+  (symbol (lib_id "LibraryAudioBoard:SJ-3523-SMT-TR") (at 62.23 115.57 0) (unit 1)
+    (in_bom yes) (on_board yes) (fields_autoplaced)
+    (property "Reference" "J4" (id 0) (at 62.23 105.41 0))
+    (property "Value" "SJ-3523-SMT-TR" (id 1) (at 62.23 107.95 0))
+    (property "Footprint" "LibraryAudioBoard:CUI_SJ-3523-SMT-TR" (id 2) (at 63.5 109.22 0)
+      (effects (font (size 1.27 1.27)) (justify bottom) hide)
+    )
+    (property "Datasheet" "" (id 3) (at 62.23 115.57 0)
+      (effects (font (size 1.27 1.27)) hide)
+    )
+    (property "Mfr" "CUI Inc" (id 4) (at 62.23 115.57 0)
+      (effects (font (size 1.27 1.27)) (justify bottom) hide)
+    )
+    (pin "1")
+    (pin "2")
+    (pin "3")
+  )
   (symbol (lib_id "Connector_Generic:Conn_01x02") (at 95.25 102.87 0) (mirror y) (unit 1)

Commit message: Update the PCB routing
Other:
- moved on the sheet: C13, C15, C17, R10, R12, R13
