File: hardware/AUDIO-BOARD.kicad_pcb (KiCad board)
At the start: 2 copper layers, 66 x 46 mm, 79 parts, among them J1 CON_USB_GCT_USB4105_REVA, J3 CON_USB_GCT_USB4105_REVA, J4 BATT, J5 SD-CARD-MEM2051-00-195-00-A, M1 MNT, M2 MNT, M3 MNT, M4 MNT, Q1 DMP2040USD-13, Q2 DMP2040USD-13, Q3 SI2324DS-T1-GE3, Q4 SI2324DS-T1-GE3, SW1 RST, U1 CS42L51-CNZ, U2 TLV73333PDBV, U3 STM32H725ZET6, U4 MCP73831-2-OT, Y1 12MHz

Commit message: update the design
Parts:
- added L1: 39n, Inductor_SMD:L_0603_1608Metric, F.Cu at (162.0, 98.5)
- C6, C7: value 100n -> 1u(X7R)
- Y1: value 12MHz -> 8MHz
- moved Y1 32.7 mm to (124.5, 81.5), turned to 0 degrees
Connections:
- C25 pad 1: Net-(C25-Pad1) -> /XIN
- C33 pad 1: Net-(C33-Pad1) -> /XOUT
- C6 pad 1: +3.3V -> Net-(C6-Pad1)
- C6 pad 2: GND -> Net-(C6-Pad2)
- C7 pad 1: +3.3V -> Net-(C7-Pad1)
- U3 pad 25: Net-(C33-Pad1) -> /XIN
- U3 pad 26: Net-(C25-Pad1) -> /XOUT
- Y1 pad 1: XIN -> /XIN
- Y1 pad 2: GND -> Net-(Y1-Pad2)
- Y1 pad 3: XOUT -> /XOUT
- Y1 pad 4: GND -> Net-(Y1-Pad2)

Commit message: update the design
Parts:
- removed C36, C38, C39, C40: 100n, Capacitor_SMD:C_0603_1608Metric
- removed C37: 2.2u, Capacitor_SMD:C_0603_1608Metric
- removed C41, C42: 10u, Capacitor_SMD:C_0805_2012Metric
- removed L1: 39n, Inductor_SMD:L_0603_1608Metric
- added J2: STLINK, Connector_PinHeader_2.54mm:PinHeader_1x04_P2.54mm_Vertical, F.Cu at (138.5, 91.5)
- added J6: CON_USB_GCT_USB4105_REVA, 1KiCadLib:CON_USB_GCT_USB4105_REVA, F.Cu at (165.5, 84.8)
- added J7: BATT, Connector_JST:JST_EH_S2B-EH_1x02_P2.50mm_Horizontal, F.Cu at (155.5, 86.2)
- added R20: 10K, Resistor_SMD:R_0805_2012Metric, F.Cu at (107.2, 121.6)
- added R21: 10K, Resistor_SMD:R_0805_2012Metric, F.Cu at (107.2, 124.6)
- added U5: MCP73831-2-OT, Package_TO_SOT_SMD:SOT-23-5, F.Cu at (117.8, 114.0)
- added U6: TLV73333PDBV, Package_TO_SOT_SMD:SOT-23-5, F.Cu at (149.0, 63.2)
- added U7: NCP163ASN250T1G, Package_TO_SOT_SMD:SOT-23-5, F.Cu at (112.7, 114.0)
- C1: value 22p -> 12p
- C10, C11, C9: value 1u -> 100n; footprint Capacitor_SMD:C_0805_2012Metric -> Capacitor_SMD:C_0603_1608Metric
- C13: value 10u -> 22p; footprint Capacitor_SMD:C_0805_2012Metric -> Capacitor_SMD:C_0603_1608Metric
- C14: value 100n -> 22p
- C15, C22, C23: value 100n -> 1u; footprint Capacitor_SMD:C_0603_1608Metric -> Capacitor_SMD:C_0805_2012Metric
- C16: value 100n -> 150p
- C17: value 10u -> 150p; footprint Capacitor_SMD:C_0805_2012Metric -> Capacitor_SMD:C_0603_1608Metric
- C18: value 10u -> 1u(X7R); footprint Capacitor_SMD:C_0805_2012Metric -> Capacitor_SMD:C_0603_1608Metric
- C19: value 100n -> 1u(X7R); footprint Capacitor_SMD:C_0201_0603Metric -> Capacitor_SMD:C_0603_1608Metric
- C2: value 22p -> 100n
- C20: value 4.7u -> 100n; footprint Capacitor_SMD:C_0805_2012Metric -> Capacitor_SMD:C_0603_1608Metric
- C21: value 100n -> 1u
- C25, C33: value 12p -> 10u; footprint Capacitor_SMD:C_0603_1608Metric -> Capacitor_SMD:C_0805_2012Metric
- C29, C30, C31, C32, C34: value 100n -> 10u; footprint Capacitor_SMD:C_0603_1608Metric -> Capacitor_SMD:C_0805_2012Metric
- C3: value 1u -> 12p; footprint Capacitor_SMD:C_0805_2012Metric -> Capacitor_SMD:C_0603_1608Metric
- C35: footprint Capacitor_SMD:C_0603_1608Metric -> Capacitor_SMD:C_0201_0603Metric
- C4: value 150p -> 4.7u; footprint Capacitor_SMD:C_0603_1608Metric -> Capacitor_SMD:C_0805_2012Metric
- C5: value 150p -> 100n
- C6, C7: value 1u(X7R) -> 100n
- J3: value CON_USB_GCT_USB4105_REVA -> SD-CARD-MEM2051-00-195-00-A; footprint 1KiCadLib:CON_USB_GCT_USB4105_REVA -> 1KiCadLib:SD-CARD-MEM2051-00-195-00-A; moved to B.Cu
- J4: value BATT -> AudioJack3_Ground; footprint Connector_JST:JST_EH_S2B-EH_1x02_P2.50mm_Horizontal -> Connector_Audio:Jack_3.5mm_CUI_SJ-3523-SMT_Horizontal
- J5: value SD-CARD-MEM2051-00-195-00-A -> MIC; footprint 1KiCadLib:SD-CARD-MEM2051-00-195-00-A -> Connector_PinSocket_2.54mm:PinSocket_1x02_P2.54mm_Vertical
- R1, R2: value 51R -> 10K
- R10, R11: value 10K -> 51R
- R13: value 10K -> 100R
- R15: value 10K -> 2K
- R16, R17, R18: value 10K -> 100K
- R19: value 2K -> 330R
- R3: value 100R -> 10K
- R5, R6, R7: value 100K -> 10K
- R8: value 330R -> 10K
- U1: value CS42L51-CNZ -> STM32F446RETx; footprint Package_DFN_QFN:QFN-32-1EP_5x5mm_P0.5mm_EP3.1x3.1mm -> Package_QFP:LQFP-64_10x10mm_P0.5mm
- U2: value TLV73333PDBV -> D-ESD-PESD2ETH-AD; footprint Package_TO_SOT_SMD:SOT-23-5 -> Package_TO_SOT_SMD:SOT-23-6
- U3: value STM32H725ZET6 -> TSOP38G36; footprint Package_QFP:LQFP-144_20x20mm_P0.5mm -> OptoDevice:Vishay_MINICAST-3Pin
- U4: value MCP73831-2-OT -> CS42L51-CNZ; footprint Package_TO_SOT_SMD:SOT-23-5 -> Package_DFN_QFN:QFN-32-1EP_5x5mm_P0.5mm_EP3.1x3.1mm
- moved U4 112.1 mm to (118.5, 72.8)
- moved Q2 59.1 mm to (155.2, 74.5)
- moved SW1 53.3 mm to (146.5, 56.8)
- moved C22 51.1 mm to (118.0, 78.0)
- moved C24 48.0 mm to (126.5, 77.0)
- moved Q1 47.1 mm to (155.2, 80.2)
- moved J3 30.2 mm to (122.2, 62.5), turned to 180 degrees
- moved J5 27.8 mm to (138.5, 56.3)
- moved U1 24.4 mm to (139.0, 71.8), turned to 180 degrees
- moved Y1 24.2 mm to (147.4, 73.8), turned to 90 degrees
- moved U3 20.8 mm to (130.2, 89.5)
- moved J4 4.94 mm to (115.8, 84.8), turned to 90 degrees
- moved J1 2.00 mm to (165.0, 63.0)
Connections:
- C1 pad 1: Net-(C1-Pad1) -> /XOUT
- C1 pad 2: Net-(C1-Pad2) -> GND
- C10 pad 1: +2V5 -> +3.3V
- C11 pad 1: Net-(C11-Pad1) -> +3.3V
- C12 pad 1: +2V5 -> +3.3V
- C13 pad 2: GND -> Net-(C13-Pad2)
- C14 pad 1: +2V5 -> Net-(C14-Pad1)
- C14 pad 2: GND -> Net-(C14-Pad2)
- C15 pad 1: +2V5 -> Net-(C15-Pad1)
- C15 pad 2: GND -> Net-(C15-Pad2)
- C16 pad 1: +2V5 -> Net-(C16-Pad1)
- C17 pad 1: /PowerSupply/DC_OUT -> Net-(C17-Pad1)
- C18 pad 1: +3.3V -> Net-(C18-Pad1)
- C18 pad 2: GND -> Net-(C18-Pad2)
- C2 pad 2: Net-(C2-Pad2) -> GND
- C20 pad 1: Net-(C20-Pad1) -> +3.3V
- C21 pad 1: Net-(C20-Pad1) -> Net-(C21-Pad1)
- C22 pad 1: +3.3V -> +2V5
- C23 pad 1: +3.3V -> Net-(C23-Pad1)
- C24 pad 1: +3.3V -> +2V5
- C25 pad 1: /XIN -> Net-(C25-Pad1)
- C26 pad 1: +3.3V -> +2V5
- C27 pad 1: +3.3V -> +2V5
- C28 pad 1: +3.3V -> +2V5
- C29 pad 1: Net-(C29-Pad1) -> VBUS
- C3 pad 1: unconnected-(C3-Pad1) -> /XIN
- C3 pad 2: Net-(C3-Pad2) -> GND
- C30 pad 1: +3.3V -> +BATT
- C31 pad 1: +3.3V -> /PowerSupply/DC_OUT
- C32 pad 1: +3.3V -> /PowerSupply/DC_OUT
- C33 pad 1: /XOUT -> +3.3V
- C34 pad 1: +3.3V -> +2V5
- C5 pad 1: Net-(C5-Pad1) -> +3.3V
- C6 pad 1: Net-(C6-Pad1) -> +3.3V
- C6 pad 2: Net-(C6-Pad2) -> GND
- C7 pad 1: Net-(C7-Pad1) -> +3.3V
- C9 pad 1: Net-(C9-Pad1) -> +3.3V
- J1 pad A4/B9: Net-(J1-PadA4/B9) -> /USB_POWER
- J1 pad A6: unconnected-(J1-PadA6) -> USB+
- J1 pad A7: unconnected-(J1-PadA7) -> USB-
- J1 pad B4/A9: Net-(J1-PadA4/B9) -> /USB_POWER
- J1 pad B6: unconnected-(J1-PadB6) -> USB+
- J1 pad B7: unconnected-(J1-PadB7) -> USB-
- J5 pad 1: SD_D2 -> Net-(C15-Pad1)
- J5 pad 2: SD_D3 -> GND
- Q4 pad 1: Net-(C19-Pad1) -> Net-(C35-Pad1)
- R1 pad 1: Net-(C1-Pad2) -> +3.3V
- R1 pad 2: GND -> Net-(C2-Pad1)
- R10 pad 1: Net-(Q2-Pad1) -> Net-(C13-Pad2)
- R10 pad 2: Net-(Q2-Pad2) -> GND
- R11 pad 1: Net-(R11-Pad1) -> Net-(C14-Pad2)
- R12 pad 1: +3.3V -> GND
- R12 pad 2: Net-(R12-Pad2) -> CODEC_M/~{S}
- R13 pad 1: +3.3V -> Net-(C15-Pad2)
- R13 pad 2: Net-(C29-Pad1) -> Net-(R13-Pad2)
- R14 pad 2: SD_CMD -> CODEC_RST
- R15 pad 1: +3.3V -> Net-(R15-Pad1)
- R15 pad 2: SD_D3 -> GND
- R16 pad 1: +3.3V -> VBUS
- R16 pad 2: SD_D2 -> Net-(C35-Pad1)
- R17 pad 1: +3.3V -> Net-(C35-Pad1)
- R17 pad 2: SD_D1 -> GND
- R18 pad 1: +3.3V -> +BATT
- R18 pad 2: SD_D0 -> Net-(Q3-Pad1)
- R19 pad 1: Net-(R19-Pad1) -> Net-(Q3-Pad1)
- R19 pad 2: GND -> Net-(Q2-Pad2)
- R2 pad 1: Net-(C2-Pad2) -> GND
- R2 pad 2: GND -> Net-(R2-Pad2)
- R3 pad 1: Net-(C3-Pad2) -> +3.3V
- R3 pad 2: Net-(R3-Pad2) -> SD_CMD_PD2
- R4 pad 2: /Audio Codec/~{RST} -> I2C_SDA_PB7
- R5 pad 1: VBUS -> +3.3V
- R5 pad 2: Net-(C19-Pad1) -> SD_D3_PC11
- R6 pad 1: Net-(C19-Pad1) -> +3.3V
- R6 pad 2: GND -> I2C_SCL_PB6
- R7 pad 1: +BATT -> +3.3V
- R7 pad 2: Net-(Q3-Pad1) -> SD_D2_PB1
- R8 pad 1: Net-(Q3-Pad1) -> +3.3V
- R8 pad 2: Net-(Q2-Pad2) -> SD_D1_PB0
- R9 pad 1: Net-(Q1-Pad1) -> +3.3V
- R9 pad 2: Net-(Q1-Pad2) -> SD_D0_PC8
- SW1 pad 1: Net-(C29-Pad1) -> Net-(C2-Pad1)
- U1 pad 1: /Audio Codec/SCL -> +3.3V
- U1 pad 10: Net-(C1-Pad1) -> unconnected-(U1-Pad10)
- U1 pad 11: Net-(C2-Pad1) -> unconnected-(U1-Pad11)
- U1 pad 12: +2V5 -> GND
- U1 pad 13: GND -> +3.3V
- U1 pad 14: Net-(C11-Pad1) -> unconnected-(U1-Pad14)
- U1 pad 15: Net-(C9-Pad1) -> unconnected-(U1-Pad15)
- U1 pad 16: Net-(C13-Pad1) -> unconnected-(U1-Pad16)
- U1 pad 18: unconnected-(U1-Pad18) -> GND
- U1 pad 19: unconnected-(U1-Pad19) -> +3.3V
- U1 pad 2: /Audio Codec/SDA -> unconnected-(U1-Pad2)
- U1 pad 20: unconnected-(U1-Pad20) -> I2S_WS_PA4
- U1 pad 21: Net-(C4-Pad1) -> I2S_SCLK_PA5
- U1 pad 22: Net-(C5-Pad1) -> unconnected-(U1-Pad22)
- U1 pad 23: Net-(R3-Pad2) -> I2S_DIN_PA7
- U1 pad 24: Net-(R3-Pad2) -> I2S_MCLK_PC4
- U1 pad 25: /Audio Codec/~{RST} -> unconnected-(U1-Pad25)
- U1 pad 26: +3.3V -> SD_D1_PB0
- U1 pad 27: +2V5 -> SD_D2_PB1
- U1 pad 28: GND -> SD_CLK_PB2
- U1 pad 29: /Audio Codec/SDOUT -> unconnected-(U1-Pad29)
- U1 pad 3: /Audio Codec/SCL -> unconnected-(U1-Pad3)
- U1 pad 30: /Audio Codec/MCLK -> Net-(C4-Pad1)
- U1 pad 31: /Audio Codec/SCLK -> GND
- U1 pad 32: /Audio Codec/SDIN -> +3.3V
- U1 pad 33: GND -> unconnected-(U1-Pad33)
- U1 pad 4: GND -> unconnected-(U1-Pad4)
- U1 pad 5: +2V5 -> /XIN
- U1 pad 6: Net-(C6-Pad1) -> /XOUT
- U1 pad 7: GND -> Net-(C2-Pad1)
- U1 pad 8: Net-(C6-Pad2) -> unconnected-(U1-Pad8)
- U1 pad 9: Net-(C7-Pad1) -> unconnected-(U1-Pad9)
- U2 pad 1: /PowerSupply/DC_OUT -> USB_P
- U2 pad 3: /PowerSupply/DC_OUT -> USB_N
- U2 pad 4: unconnected-(U2-Pad4) -> USB-
- U2 pad 5: +3.3V -> /USB_POWER
- U3 pad 1: unconnected-(U3-Pad1) -> IRR_OUT
- U3 pad 2: unconnected-(U3-Pad2) -> GND
- U3 pad 3: unconnected-(U3-Pad3) -> +3.3V
- U4 pad 1: unconnected-(U4-Pad1) -> I2S_WS_PA4
- U4 pad 2: GND -> I2C_SDA_PB7
- U4 pad 3: +BATT -> I2C_SCL_PB6
- U4 pad 4: VBUS -> GND
- U4 pad 5: Net-(R19-Pad1) -> +2V5

Commit message: Update placements
Parts:
- removed Q1, Q2: DMP2040USD-13, Package_SO:SOIC-8_3.9x4.9mm_P1.27mm
- removed Q3, Q4: SI2324DS-T1-GE3, Package_TO_SOT_SMD:SOT-23
- added C36: 120p, Capacitor_SMD:C_0805_2012Metric, F.Cu at (134.5, 55.6)
- added C37: 22u, Capacitor_SMD:C_0805_2012Metric, F.Cu at (132.9, 58.7)
- added C38: 22u, Capacitor_SMD:C_0805_2012Metric, F.Cu at (130.7, 58.6)
- added C39: 100u, Capacitor_SMD:C_0805_2012Metric, F.Cu at (158.1, 83.6)
- added D1: LED, LED_SMD:LED_0805_2012Metric, F.Cu at (154.2, 92.3)
- added D2: D_Schottky, Diode_SMD:D_SOD-123, F.Cu at (134.7, 62.4)
- added D3: LED, LED_SMD:LED_0805_2012Metric, F.Cu at (128.5, 58.5)
- added L1: 2.2uH, Inductor_SMD:L_2010_5025Metric, F.Cu at (140.7, 62.4)
- added R22: 10K, Resistor_SMD:R_0805_2012Metric, F.Cu at (151.7, 83.6)
- added U10: TPS2116, Package_TO_SOT_SMD:SOT-23-8, F.Cu at (154.9, 83.6)
- added U8: AP22652W6-7, Package_TO_SOT_SMD:SOT-23-6, F.Cu at (143.5, 58.8)
- added U9: TPS613222ADBV, Package_TO_SOT_SMD:SOT-23-5, F.Cu at (136.4, 58.7)
- C29, C30, R15, U5: moved to B.Cu
- C35: value 100n -> 22u; footprint Capacitor_SMD:C_0201_0603Metric -> Capacitor_SMD:C_0805_2012Metric
- J4: value AudioJack3_Ground -> SJ-3523-SMT-TR; footprint Connector_Audio:Jack_3.5mm_CUI_SJ-3523-SMT_Horizontal -> LibraryAudioBoard:CUI_SJ-3523-SMT-TR
- J7: footprint Connector_JST:JST_EH_S2B-EH_1x02_P2.50mm_Horizontal -> Connector_JST:JST_EH_B2B-EH-A_1x02_P2.50mm_Vertical
- R16: value 100K -> 1K; moved to B.Cu
- R17: value 100K -> 20k
- R18: value 100K -> 5R; footprint Resistor_SMD:R_0805_2012Metric -> Diode_SMD:D_0805_2012Metric
- R19: value 330R -> 10K
- R21: value 10K -> 1K
- moved C11 90.4 mm to (128.7, 86.8), turned to 180 degrees
- moved R3 90.4 mm to (120.8, 59.0), turned to -90 degrees
- moved C12 84.2 mm to (115.9, 64.0)
- moved R7 82.2 mm to (116.5, 59.0), turned to -90 degrees
- moved R5 80.7 mm to (118.6, 59.0), turned to -90 degrees
- moved C14 80.5 mm to (112.6, 75.5), turned to -90 degrees
- moved C13 77.7 mm to (117.9, 67.3), turned to 90 degrees
- moved C18 76.7 mm to (117.2, 70.8)
- moved R9 76.1 mm to (123.0, 59.0), turned to -90 degrees
- moved C16 74.6 mm to (121.3, 79.1), turned to -90 degrees
- moved C7 74.4 mm to (131.9, 73.7), turned to 180 degrees
- moved R21 73.0 mm to (130.9, 55.6), turned to 180 degrees
- moved R8 72.5 mm to (125.2, 59.0), turned to -90 degrees
- moved R10 72.3 mm to (116.1, 67.5), turned to -90 degrees
- moved C19 71.5 mm to (117.2, 72.4), turned to 180 degrees
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Connections:
- net /PowerSupply/DC_OUT renamed /PowerSupply/MAIN_PWR
- C35 pad 1: Net-(C35-Pad1) -> /PowerSupply/BOOST_IN
- R16 pad 1: VBUS -> +3.3V
- R16 pad 2: Net-(C35-Pad1) -> Net-(D1-Pad2)
- R17 pad 1: Net-(C35-Pad1) -> Net-(R17-Pad1)
- R18 pad 1: +BATT -> Net-(D2-Pad2)
- R18 pad 2: Net-(Q3-Pad1) -> Net-(C36-Pad1)
- R19 pad 1: Net-(Q3-Pad1) -> VBUS
- R19 pad 2: Net-(Q2-Pad2) -> Net-(R19-Pad2)
- R20 pad 1: Net-(Q1-Pad1) -> Net-(R19-Pad2)
- R20 pad 2: Net-(Q1-Pad2) -> GND
- R21 pad 1: Net-(Q2-Pad1) -> /USB_OTG_VBUS
- R21 pad 2: Net-(Q2-Pad2) -> Net-(D3-Pad2)
- U1 pad 33: unconnected-(U1-Pad33) -> /USB_OTG_EN
- U1 pad 36: unconnected-(U1-Pad36) -> IRR_OUT

Commit message: Update the PCB routing
Parts:
- added J8: TFT TOUCH SCREEN, Connector_PinSocket_2.54mm:PinSocket_1x14_P2.54mm_Vertical, F.Cu at (108.7, 59.9)
- C29, C30, J3, R15, R16, U5: moved to F.Cu
- moved J2 42.4 mm to (173.6, 81.4), turned to 180 degrees
- moved R21 36.2 mm to (167.0, 53.6), turned to 90 degrees
- moved J5 35.8 mm to (128.1, 98.2), turned to 90 degrees
- moved D3 35.6 mm to (163.6, 52.7), turned to 0 degrees
- moved C38 33.1 mm to (163.6, 55.0), turned to 180 degrees
- moved C36 32.7 mm to (167.1, 57.9), turned to 90 degrees
- moved C12 30.8 mm to (145.5, 55.4), turned to -90 degrees
- moved C37 30.7 mm to (163.5, 57.2), turned to 180 degrees
- moved R18 29.8 mm to (167.1, 62.0), turned to 90 degrees
- moved U9 27.2 mm to (163.5, 60.5), turned to 90 degrees
- moved R17 25.9 mm to (166.8, 67.9), turned to 90 degrees
- moved D2 24.9 mm to (159.3, 58.7), turned to -90 degrees
- moved C35 24.1 mm to (163.4, 64.2), turned to 0 degrees
- moved R6 22.7 mm to (158.8, 78.8)
- moved R4 22.7 mm to (158.8, 76.8)
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Connections:
- J1 pad A4/B9: /USB_POWER -> /USB_OTG_VBUS
- J1 pad B4/A9: /USB_POWER -> /USB_OTG_VBUS
- U1 pad 10: unconnected-(U1-Pad10) -> SPI2_MISO_PC2
- U1 pad 2: unconnected-(U1-Pad2) -> SPI3_nCS_PC13
- U1 pad 29: unconnected-(U1-Pad29) -> SPI2_SCK_PB10
- U1 pad 3: unconnected-(U1-Pad3) -> LCD_RST_PC14
- U1 pad 37: unconnected-(U1-Pad37) -> LCD_LED_PC6
- U1 pad 38: unconnected-(U1-Pad38) -> LCD_T_IRQ_PC7
- U1 pad 4: unconnected-(U1-Pad4) -> LCD_DC_PC15
- U1 pad 51: unconnected-(U1-Pad51) -> SPI3_SCK_PC10
- U1 pad 53: unconnected-(U1-Pad53) -> SPI3_MOSI_PC12
- U1 pad 56: unconnected-(U1-Pad56) -> SPI3_MISO_PB4
- U1 pad 62: unconnected-(U1-Pad62) -> SPI2_nCS_PB9
- U1 pad 9: unconnected-(U1-Pad9) -> SPI2_MOSI_PC1
- U2 pad 5: /USB_POWER -> /USB_OTG_VBUS
- U8 pad 3: /PowerSupply/USB_OTG_EN -> /USB_OTG_EN
Routing:
- net SPI3_MISO_PB4: track 0.00 -> 63.6 mm, vias 0 -> 3
- net SPI3_nCS_PC13: track 0.00 -> 63.4 mm, vias 0 -> 3
- net SPI3_MOSI_PC12: track 0.00 -> 60.8 mm, vias 0 -> 3
- net LCD_LED_PC6: track 0.00 -> 60.6 mm, vias 0 -> 1
- net SPI2_MISO_PC2: track 0.00 -> 59.9 mm, vias 0 -> 3
- net SPI3_SCK_PC10: track 0.00 -> 57.2 mm, vias 0 -> 3
- net SPI2_MOSI_PC1: track 0.00 -> 56.3 mm, vias 0 -> 1
- net SD_D3_PC11: track 0.00 -> 55.4 mm, vias 0 -> 2
- net /USB_OTG_VBUS: track 0.00 -> 55.4 mm, vias 0 -> 4
- net SD_D0_PC8: track 0.00 -> 54.8 mm, vias 0 -> 2
- net LCD_DC_PC15: track 0.00 -> 53.6 mm, vias 0 -> 1
- net SPI2_SCK_PB10: track 0.00 -> 53.6 mm, vias 0 -> 2
- net SD_CMD_PD2: track 0.00 -> 52.7 mm, vias 0 -> 2
- net SPI2_nCS_PB9: track 0.00 -> 49.8 mm, vias 0 -> 1
- net LCD_RST_PC14: track 0.00 -> 49.2 mm, vias 0 -> 1
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- added copper zone on F.Cu, net +2V5
- added copper zone on In2.Cu, net +2V5
- added copper zone on F.Cu, net +3.3V
- added copper zone on In2.Cu, net +3.3V
- added copper zone on F.Cu, net /PowerSupply/MAIN_PWR
- added copper zone on In2.Cu, net /PowerSupply/MAIN_PWR
- added copper zone on B.Cu, net GND
- added copper zone on F.Cu, net GND
- added copper zone on In1.Cu, net GND
- added copper zone on F.Cu, net VBUS
Other:
- board size 66 x 46 mm -> 80 x 56 mm
- copper layers 2 -> 4
